File: HARDWARE/HydroScan_V1.kicad_sch (KiCad schematic)
At the start: 138 parts, among them CN1 DB128V-5.08-2P-GN-S, J1 BATERY, Q13 2n3904S-RTK/PS_C18536, Q14 2n3904S-RTK/PS_C18536, Q15 2n3904S-RTK/PS_C18536, Q16 2n3904S-RTK/PS_C18536, SW2 BOOT, SW4 RESET, U1 IP2312-4V35, U13 ESP32-WROOM-32D, U14 CH340C, U15 CH340C, U16 ESP32-WROOM-32D, U2 BQ25798RQMR, U7 LM2576HVS-3.3

Commit message: Integrate ESP32
Parts:
- renumbered BOOT to BOOT1, RESET to RESET1
Changed lines of the file:
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@@
 		(dnp no)
 		(fields_autoplaced yes)
-		(property "Reference" "RESET"
+		(property "Reference" "RESET1"
 			(at 113.03 88.9 0)
 			(hide yes)
@@
 			(project "HydroScan_V1"
 				(path "/5017cb5d-eb32-4723-8271-7ee6dfdf0b58"
-					(reference "RESET")
+					(reference "RESET1")
 					(unit 1)
 				)
@@
 		(dnp no)
 		(fields_autoplaced yes)
-		(property "Reference" "BOOT"
+		(property "Reference" "BOOT1"
 			(at 114.3 139.7 0)
 			(hide yes)
@@
 			(project "HydroScan_V1"
 				(path "/5017cb5d-eb32-4723-8271-7ee6dfdf0b58"
-					(reference "BOOT")
+					(reference "BOOT1")
 					(unit 1)
 				)

Commit message: Aclaracion de avances
Other:
- note added: "HYDROSCAN_V1"
- note added: "Nota problemas: /Comunicacion /Alimentacion /bateria"
- note added: "Nota: Barra indicado nivel de bateria. indicador de latidos, aun no esta definido."
- note added: "Pantalla"
- note added: "Pantalla info"
- note added: "Periferia Botones"
- note removed: "SPLORATION_SEAN"
- moved on the sheet: PH_sensor1
Changed lines of the file:
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@@
 	(rectangle
 		(start 179.07 229.87)
-		(end 257.81 283.21)
+		(end 259.08 283.21)
 		(stroke
 			(width 0)
@@
 	(rectangle
 		(start 179.07 219.71)
-		(end 257.81 229.87)
+		(end 259.08 229.87)
 		(stroke
 			(width 0)
@@
 	(rectangle
 		(start 440.69 63.5)
-		(end 509.27 194.31)
+		(end 509.27 154.94)
 		(stroke
 			(width 0)
@@
 	)
 	(rectangle
-		(start 257.81 219.71)
+		(start 259.08 219.71)
 		(end 336.55 229.87)
 		(stroke
@@
 	)
 	(rectangle
+		(start 440.69 320.04)
+		(end 610.87 424.18)
+		(stroke
+			(width 0)
+			(type default)
+		)
+		(fill
+			(type none)
+		)
+	)
+	(rectangle
 		(start 511.81 77.47)
 		(end 612.14 154.94)
@@
 	(rectangle
 		(start 17.78 64.77)
-		(end 257.81 218.44)
+		(end 256.54 218.44)
 		(stroke
 			(width 0.0762)
@@
 	)
 	(rectangle
-		(start 257.81 229.87)
+		(start 259.08 229.87)
 		(end 336.55 283.21)
 		(stroke
@@
 	)
 	(rectangle
+		(start 440.69 424.18)
+		(end 610.87 528.32)
+		(stroke
+			(width 0)
+			(type default)
+		)
+		(fill
+			(type none)
+		)
+	)
+	(rectangle
 		(start 697.23 66.04)
 		(end 756.92 154.94)
@@
 	)
 	(rectangle
-		(start 181.61 67.31)
+		(start 179.07 67.31)
 		(end 256.54 77.47)
 		(stroke
@@
 		)
 	)
+	(text "Periferia Botones"
+		(exclude_from_sim no)
+		(at 516.636 434.086 0)
+		(effects
+			(font
+				(size 6.35 6.35)
+				(thickness 1.27)
+				(bold yes)
+			)
+		)
+	)
 	(text "MOTOR__DRIVER"
 		(exclude_from_sim no)
@@
 		)
 	)
-	(text "SPLORATION_SEAN\n"
+	(text "HYDROSCAN_V1"
 		(exclude_from_sim no)
-		(at 195.58 30.48 0)
+		(at 207.772 33.274 0)
 		(effects
 			(font
@@
 		)
 	)
+	(text "Nota:\nBarra indicado nivel de bateria.\nindicador de latidos, aun no esta definido.\n"
+		(exclude_from_sim no)
+		(at 445.77 353.314 0)
+		(effects
+			(font
+				(size 2.286 2.286)
+				(thickness 0.1588)
+			)
+			(justify left)
+		)
+	)
 	(text "COMPLICADO\n"
 		(exclude_from_sim no)
@@
 		)
 	)
+	(text "Pantalla info"
+		(exclude_from_sim no)
+		(at 476.504 340.106 0)
+		(effects
+			(font
+				(size 6.35 6.35)
+				(thickness 1.27)
+				(bold yes)
+			)
+		)
+	)
 	(text "CARGADOR_BAT 14.2V"
 		(exclude_from_sim no)
@@
 		)
 	)
+	(text "Pantalla"
+		(exclude_from_sim no)
+		(at 517.144 326.644 0)
+		(effects
+			(font
+				(size 6.35 6.35)
+				(thickness 1.27)
+				(bold yes)
+			)
+		)
+	)
 	(text "Cerebro"
 		(exclude_from_sim no)
@@
 		)
 	)
+	(text "Nota problemas:\n/Comunicacion\n/Alimentacion \n/bateria"
+		(exclude_from_sim no)
+		(at 326.136 166.878 0)
+		(effects
+			(font
+				(size 2.286 2.286)
+				(thickness 0.1588)
+			)
+			(justify left)
+		)
+	)
 	(text "AMBU"
 		(exclude_from_sim no)
@@
 	(wire
 		(pts
+			(xy 781.05 153.67) (xy 778.51 153.67)
+		)
+		(stroke
+			(width 0)
+			(type default)
+		)
+	)
+	(wire
+		(pts
 			(xy 744.22 255.27) (xy 755.65 255.27)
 		)
@@
 	(symbol
 		(lib_id "Mis_creaciones:PH-4502C")
-		(at 54.61 247.65 0)
+		(at 55.88 243.84 0)
 		(unit 1)
 		(body_style 1)
@@
 		(fields_autoplaced yes)
 		(property "Reference" "PH_sensor1"
-			(at 56.515 243.84 0)
+			(at 57.785 240.03 0)
 			(show_name no)
 			(do_not_autoplace no)
@@
 		)
 		(property "Value" "PH-4502C"
-			(at 56.515 246.38 0)
+			(at 57.785 242.57 0)
 			(show_name no)
 			(do_not_autoplace no)
@@
 		)
 		(property "Footprint" ""
-			(at 54.61 247.65 0)
+			(at 55.88 243.84 0)
 			(hide yes)
 			(show_name no)
@@
 		)
 		(property "Datasheet" ""
-			(at 54.61 247.65 0)
+			(at 55.88 243.84 0)
 			(hide yes)
 			(show_name no)
@@
 		)
 		(property "Description" ""
-			(at 54.61 247.65 0)
+			(at 55.88 243.84 0)
 			(hide yes)
 			(show_name no)
@@
 	(symbol
 		(lib_id "power:GND")
-		(at 778.51 153.67 90)
+		(at 781.05 153.67 90)
 		(mirror x)
 		(unit 1)
@@
 		(dnp no)
 		(property "Reference" "#PWR0145"
-			(at 784.86 153.67 0)
+			(at 787.4 153.67 0)
 			(hide yes)
 			(show_name no)
@@
 		)
 		(property "Value" "GND"
-			(at 783.59 153.67 90)
+			(at 786.13 153.67 90)
 			(show_name no)
 			(do_not_autoplace no)
@@
 		)
 		(property "Footprint" ""
-			(at 778.51 153.67 0)
+			(at 781.05 153.67 0)
 			(hide yes)
 			(show_name no)
@@
 		)
 		(property "Datasheet" ""
-			(at 778.51 153.67 0)
+			(at 781.05 153.67 0)
 			(hide yes)
 			(show_name no)
@@
 		)
 		(property "Description" "Power symbol creates a global label with name \"GND\" , ground"
-			(at 778.51 153.67 0)
+			(at 781.05 153.67 0)
 			(hide yes)
 			(show_name no)

Commit message: Avances puerto USB C
Parts:
- removed D32, D33, D34: LESD5D5.0CT1G, EasyEDA:SOD-523_L1.2-W0.8-LS1.6-BI, symbol EasyEDA:LESD5D5.0CT1G
- added D1, D4: SM05.TCT, EasyEDA:SOT-23-3_L2.9-W1.3-P0.95-LS2.4-BR, symbol EasyEDA:SM05.TCT
- C22, C23: footprint PCM_Capacitor_SMD_AKL:C_0805_2012Metric_Pad1.18x1.45mm_HandSolder -> Capacitor_SMD:C_0805_2012Metric_Pad1.18x1.45mm_HandSolder
- R84, R85: footprint PCM_Resistor_SMD_AKL:R_0805_2012Metric_Pad1.20x1.40mm_HandSolder -> Capacitor_SMD:C_0805_2012Metric_Pad1.18x1.45mm_HandSolder
Connections:
- net CC1_1: now also D1.2
- net CC2_1: now also D4.1
- net GND: now also D1.3, D4.3
- net V5_1: now also D1.1, D4.2
Other:
- note added: "Resistencio de detencion"
- note added: "proteccion TVS"
- moved on the sheet: D23, R83

Commit message: change 2
Parts:
- removed D23: 1N5819HW-7-F, EasyEDA:SOD-123_L2.7-W1.6-LS3.7-RD, symbol EasyEDA:1N5819HW-7-F
- added D5: SS54_C22452, EasyEDA:SMA_L4.4-W2.8-LS5.4-R-RD, symbol EasyEDA:SS54_C22452
- R13, R83: footprint PCM_Resistor_SMD_AKL:R_0805_2012Metric_Pad1.20x1.40mm_HandSolder -> Capacitor_SMD:C_0805_2012Metric_Pad1.18x1.45mm_HandSolder
Connections:
- net 5V+: now also D5.2 (K)
- net V5_1: now also D5.1 (A)
Changed lines of the file:
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@@
 	(wire
 		(pts
+			(xy 595.63 129.54) (xy 600.71 129.54)
+		)
+		(stroke
+			(width 0)
+			(type default)
+		)
+	)
+	(wire
+		(pts
 			(xy 764.54 288.29) (xy 770.89 288.29)
 		)
@@
 	(wire
 		(pts
+			(xy 580.39 129.54) (xy 585.47 129.54)
+		)
+		(stroke
+			(width 0)
+			(type default)
+		)
+	)
+	(wire
+		(pts
 			(xy 793.75 130.81) (xy 801.37 130.81)
 		)
@@
 	(wire
 		(pts
-			(xy 567.69 107.95) (xy 577.85 107.95)
-		)
-		(stroke
-			(width 0)
-			(type default)
-		)
-	)
-	(wire
-		(pts
 			(xy 113.03 133.35) (xy 121.92 133.35)
 		)
@@
 	(wire
 		(pts
-			(xy 588.01 107.95) (xy 593.09 107.95)
-		)
-		(stroke
-			(width 0)
-			(type default)
-		)
-	)
-	(wire
-		(pts
 			(xy 698.5 283.21) (xy 702.31 283.21)
 		)
@@
 	)
 	(label "V5_1"
-		(at 567.69 107.95 0)
+		(at 580.39 129.54 0)
 		(effects
 			(font
@@
 			)
 		)
-		(property "Footprint" "PCM_Resistor_SMD_AKL:R_0805_2012Metric_Pad1.20x1.40mm_HandSolder"
+		(property "Footprint" "Capacitor_SMD:C_0805_2012Metric_Pad1.18x1.45mm_HandSolder"
 			(at 525.018 140.97 90)
 			(hide yes)
@@
 	)
 	(symbol
-		(lib_id "EasyEDA:1N5819HW-7-F")
-		(at 588.01 110.49 180)
-		(unit 1)
-		(body_style 1)
-		(exclude_from_sim no)
-		(in_bom yes)
-		(on_board yes)
-		(in_pos_files yes)
-		(dnp no)
-		(property "Reference" "D23"
-			(at 582.676 105.664 0)
-			(show_name no)
-			(do_not_autoplace no)
-			(effects
-				(font
-					(size 1.27 1.27)
-				)
-			)
-		)
-		(property "Value" "1N5819HW-7-F"
-			(at 578.866 102.87 0)
-			(show_name no)
-			(do_not_autoplace no)
-			(effects
-				(font
-					(size 1.27 1.27)
-				)
-			)
-		)
-		(property "Footprint" "EasyEDA:SOD-123_L2.7-W1.6-LS3.7-RD"
-			(at 588.01 100.33 0)
-			(hide yes)
-			(show_name no)
-			(do_not_autoplace no)
-			(effects
-				(font
-					(size 1.27 1.27)
-				)
-			)
-		)
-		(property "Datasheet" "https://lcsc.com/product-detail/Schottky-Barrier-Diodes-SBD_DIODES_1N5819HW-7-F_1N5819HW-7-F_C82544.html"
-			(at 588.01 97.79 0)
-			(hide yes)
-			(show_name no)
-			(do_not_autoplace no)
-			(effects
-				(font
-					(size 1.27 1.27)
-				)
-			)
-		)
-		(property "Description" ""
-			(at 588.01 110.49 0)
-			(hide yes)
-			(show_name no)
-			(do_not_autoplace no)
-			(effects
-				(font
-					(size 1.27 1.27)
-				)
-			)
-		)
-		(property "LCSC Part" "C82544"
-			(at 588.01 95.25 0)
-			(hide yes)
-			(show_name no)
-			(do_not_autoplace no)
-			(effects
-				(font
-					(size 1.27 1.27)
-				)
-			)
-		)
-		(pin "2"
-		)
-		(pin "1"
-		)
-		(instances
-			(project "HydroScan_V1"
-				(path "/5017cb5d-eb32-4723-8271-7ee6dfdf0b58"
-					(reference "D23")
-					(unit 1)
-				)
-			)
-		)
-	)
-	(symbol
 		(lib_id "power:GND")
 		(at 736.6 146.05 0)
@@
 			)
 		)
-		(property "Footprint" "PCM_Resistor_SMD_AKL:R_0805_2012Metric_Pad1.20x1.40mm_HandSolder"
+		(property "Footprint" "Capacitor_SMD:C_0805_2012Metric_Pad1.18x1.45mm_HandSolder"
 			(at 536.448 140.97 90)
 			(hide yes)
@@
 	(symbol
 		(lib_id "power:+5V")
-		(at 593.09 107.95 0)
+		(at 600.71 129.54 0)
 		(unit 1)
 		(body_style 1)
@@
 		(dnp no)
 		(property "Reference" "#PWR0164"
-			(at 593.09 111.76 0)
+			(at 600.71 133.35 0)
 			(hide yes)
 			(show_name no)
@@
 		)
 		(property "Value" "5V+"
-			(at 591.566 104.394 0)
+			(at 599.186 125.984 0)
 			(show_name no)
 			(do_not_autoplace no)
@@
 		)
 		(property "Footprint" ""
-			(at 593.09 107.95 0)
+			(at 600.71 129.54 0)
 			(hide yes)
 			(show_name no)
@@
 		)
 		(property "Datasheet" ""
-			(at 593.09 107.95 0)
+			(at 600.71 129.54 0)
 			(hide yes)
 			(show_name no)
@@
 		)
 		(property "Description" "Power symbol creates a global label with name \"+5V\""
-			(at 593.09 107.95 0)
+			(at 600.71 129.54 0)
 			(hide yes)
 			(show_name no)
@@
 					(unit 1)
 				)
+			)
+		)
+	)
+	(symbol
+		(lib_id "EasyEDA:SS54_C22452")
+		(at 590.55 129.54 180)
+		(unit 1)
+		(body_style 1)
+		(exclude_from_sim no)
+		(in_bom yes)
+		(on_board yes)
+		(in_pos_files yes)
+		(dnp no)
+		(fields_autoplaced yes)
+		(property "Reference" "D5"
+			(at 590.93 123.19 0)
+			(show_name no)
+			(do_not_autoplace no)
+			(effects
+				(font
+					(size 1.27 1.27)
+				)
+			)
+		)
+		(property "Value" "SS54_C22452"
+			(at 590.93 125.73 0)
+			(show_name no)
+			(do_not_autoplace no)
+			(effects
+				(font
+					(size 1.27 1.27)
+				)
+			)
+		)
+		(property "Footprint" "EasyEDA:SMA_L4.4-W2.8-LS5.4-R-RD"
+			(at 590.55 121.92 0)
+			(hide yes)
+			(show_name no)
+			(do_not_autoplace no)
+			(effects
+				(font
+					(size 1.27 1.27)
+				)
+			)
+		)
+		(property "Datasheet" "https://lcsc.com/product-detail/Schottky-Barrier-Diodes-SBD_SS54_C22452.html"
+			(at 590.55 119.38 0)
+			(hide yes)
+			(show_name no)
+			(do_not_autoplace no)
+			(effects
+				(font
+					(size 1.27 1.27)
+				)
+			)
+		)
+		(property "Description" "SS54"
+			(at 590.55 129.54 0)
+			(hide yes)
+			(show_name no)
+			(do_not_autoplace no)
+			(effects
+				(font
+					(size 1.27 1.27)
+				)
+			)
+		)
+		(property "Manufacturer" "MDD(辰达半导体)"
+			(at 590.55 116.84 0)
+			(hide yes)
+			(show_name no)
+			(do_not_autoplace no)
+			(effects
+				(font
+					(size 1.27 1.27)
+				)
+			)
+		)
+		(property "MPN" "SS54"
+			(at 590.55 114.3 0)
+			(hide yes)
+			(show_name no)
+			(do_not_autoplace no)
+			(effects
+				(font
+					(size 1.27 1.27)
+				)
+			)
+		)
+		(property "LCSC Part" "C22452"
+			(at 590.55 111.76 0)
+			(hide yes)
+			(show_name no)
+			(do_not_autoplace no)
+			(effects
+				(font
+					(size 1.27 1.27)
+				)
+			)
+		)
+		(pin "1"
+		)
+		(pin "2"
+		)
+		(instances
+			(project "HydroScan_V1"
+				(path "/5017cb5d-eb32-4723-8271-7ee6dfdf0b58"
+					(reference "D5")
+					(unit 1)
+				)

Commit message: EsP32 terminate
Parts:
- removed C21, C26: 10uf, PCM_Capacitor_SMD_AKL:C_0805_2012Metric_Pad1.18x1.45mm_HandSolder, symbol Device:C
- removed CN1: DB128V-5.08-2P-GN-S, EasyEDA:CONN-TH_2P-P5.08_DIBO_DB128V-5.08, symbol EasyEDA:DB128V-5.08-2P-GN-S
- removed D3: B330A, PCM_Diode_SMD_AKL:D_SMA, symbol PCM_Diode_Schottky_AKL:B330A
- removed D5: SS54_C22452, EasyEDA:SMA_L4.4-W2.8-LS5.4-R-RD, symbol EasyEDA:SS54_C22452
- added C51, C52: CL32B106KBJNNNE, EasyEDA:C1210, symbol EasyEDA:CL32B106KBJNNNE
- added CN2: DB128V-5.08-2P-GN-S, EasyEDA:CONN-TH_2P-P5.08_DIBO_DB128V-5.08, symbol EasyEDA:DB128V-5.08-2P-GN-S
- added D5: B330A, EasyEDA:SMA_L4.3-W2.6-LS5.1-RD, symbol EasyEDA:B330A
- added LED17: YLED0805G, EasyEDA:LED0805-FD-GREEN, symbol EasyEDA:YLED0805G
- added R22: 2.2k, Resistor_SMD:R_0805_2012Metric_Pad1.20x1.40mm_HandSolder, symbol Device:R
- C1, C14, C15, C16, C17, C18, C2, C20, C3, C39, C4, C40, C5, C6, C7, C8: footprint PCM_Capacitor_SMD_AKL:C_0805_2012Metric_Pad1.18x1.45mm_HandSolder -> Capacitor_SMD:C_0805_2012Metric_Pad1.18x1.45mm_HandSolder
- R11, R12, R18, R74, R75, R79, R81, R82: footprint PCM_Resistor_SMD_AKL:R_0805_2012Metric_Pad1.20x1.40mm_HandSolder -> Resistor_SMD:R_0805_2012Metric_Pad1.20x1.40mm_HandSolder
- R84, R85: footprint Capacitor_SMD:C_0805_2012Metric_Pad1.18x1.45mm_HandSolder -> Resistor_SMD:R_0805_2012Metric_Pad1.20x1.40mm_HandSolder
- U16: footprint RF_Module:ESP32-WROOM-32D -> RF_Module:ESP32-WROOM-32U
Connections:
- net +3.3VCC is gone; now on net 3.3V: U7.4 (Feedback)
- net +12V_F: no longer C18.1, C19.1, U7.1 (Vin)
- net 3.3V: no longer C40.1, U15.16 (VCC)
- net GND: now also C51.1, C52.1, CN2.1, D5.2 (A), LED17.2 (K)
- net SYS: now also C18.1, C19.1, U7.1 (Vin)
- net V5_1: now also C40.1, U15.16 (VCC), R22.1
- net VAC1: now also C51.2, C52.2
- net V_BATTERY__1: now also CN2.2
- net at L2.1, U7.2 (Output): now also D5.1 (C)
- net at JP4.2 (B), U2.23 (BAT): no longer U2.22 (BAT)
- new net: LED17.1 (A), R22.2
Other:
- moved on the sheet: D1, R11

Commit message: cambios en el fast charging
Parts:
- removed R13, R83: 5.11k, Capacitor_SMD:C_0805_2012Metric_Pad1.18x1.45mm_HandSolder, symbol Device:R
- added C21: 1uf, Capacitor_SMD:C_0805_2012Metric_Pad1.18x1.45mm_HandSolder, symbol Device:C
- added LED18: YLED0805G, EasyEDA:LED0805-FD-GREEN, symbol EasyEDA:YLED0805G
- added R23: 1k, Resistor_SMD:R_0805_2012Metric_Pad1.20x1.40mm_HandSolder, symbol Device:R
- added R24: 10k, Resistor_SMD:R_0805_2012Metric_Pad1.20x1.40mm_HandSolder, symbol Device:R
- added R26: 2.2k, Resistor_SMD:R_0805_2012Metric_Pad1.20x1.40mm_HandSolder, symbol Device:R
- added U3: CH224K, EasyEDA:ESSOP-10_L4.9-W3.9-P1.0-LS6.0-TL-EP, symbol EasyEDA:CH224K
- C20: footprint Capacitor_SMD:C_0805_2012Metric_Pad1.18x1.45mm_HandSolder -> Capacitor_SMD:C_0201_0603Metric
- C32: footprint PCM_Capacitor_SMD_AKL:C_0805_2012Metric_Pad1.18x1.45mm_HandSolder -> Capacitor_SMD:C_0201_0603Metric
Connections:
- net CC1_1: now also U3.7 (CC1)
- net CC2_1: now also U3.6 (CC2)
- net GND: now also C21.2, U3.11 (GND), U3.9 (CFG1)
- net V5_1: now also R23.1, R24.1; no longer U15.16 (VCC)
- new net: R24.2, U3.8 (VBUS)
- new net: LED18.1 (A), R26.2
- new net: LED18.2 (K), U3.10 (PG)
- new net VDD: C21.1, R23.2, R26.1, U3.1 (VDD), U3.2 (CFG2), U3.3 (CFG3)
Other:
- note added: "Fast chargin 15V/3A"
- note removed: "Resistencio de detencion"
- moved on the sheet: C22, C23, CN2, D1, D4, R84, R85, USB1

Commit message: USB c and Fast chargin update finish
Parts:
- removed LED18: YLED0805G, EasyEDA:LED0805-FD-GREEN, symbol EasyEDA:YLED0805G
- removed R26: 2.2k, Resistor_SMD:R_0805_2012Metric_Pad1.20x1.40mm_HandSolder, symbol Device:R
- added BT1: Battery, symbol Device:Battery
- added C26: 0.1uf, Capacitor_SMD:C_0805_2012Metric_Pad1.18x1.45mm_HandSolder, symbol Device:C
- added C53: 220nF, Capacitor_SMD:C_0805_2012Metric_Pad1.18x1.45mm_HandSolder, symbol Device:C
- added C54, C56: 10uF, Capacitor_SMD:C_0805_2012Metric_Pad1.18x1.45mm_HandSolder, symbol Device:C
- added C55, C57: 1uF, Capacitor_SMD:C_0805_2012Metric_Pad1.18x1.45mm_HandSolder, symbol Device:C
- added D3, D6: SS54_C22452, EasyEDA:SMA_L4.4-W2.8-LS5.4-R-RD, symbol EasyEDA:SS54_C22452
- added L4: SMDRI127-220MT, EasyEDA:IND-SMD_L12.3-W12.3_SMDRI127, symbol EasyEDA:SMDRI127-220MT
- added Q1: AO4435_C2944310, EasyEDA:SOP-8_L5.0-W3.8-P1.27-LS6.0-BL, symbol EasyEDA:AO4435_C2944310
- added R13: YLRY12-3-60F, EasyEDA:R2512, symbol EasyEDA:YLRY12-3-60F
- added R25: 120, Resistor_SMD:R_0805_2012Metric_Pad1.20x1.40mm_HandSolder, symbol Device:R
- added R27: 100K, PCM_Resistor_SMD_AKL:R_0805_2012Metric_Pad1.20x1.40mm_HandSolder, symbol Device:R
- added R28: 9110K, PCM_Resistor_SMD_AKL:R_0805_2012Metric_Pad1.20x1.40mm_HandSolder, symbol Device:R
- added R29: 10k, Resistor_SMD:R_0805_2012Metric_Pad1.20x1.40mm_HandSolder, symbol Device:R
- added U4: CN3795, EasyEDA:SSOP-10_L4.9-W3.9-P1.00-LS6.0-BL, symbol EasyEDA:CN3795
Connections:
- net 3.3V: now also C40.1, U15.16 (VCC), R29.2
- net GND: now also BT1.2 (-), C53.1, C54.1, C55.1, C56.1, C57.1, D3.1 (A), R27.1, U4.2 (GND)
- net IO16_1: now also U3.10 (PG), R29.1
- net V5_1: now also C54.2, C55.2, D6.1 (A), U4.9 (VCC); no longer C40.1
- new net: C26.1, U4.1 (VG)
- new net: Q1.4 (G), U4.10 (DRV)
- new net: R25.2, U4.5 (COM)
- new net: R27.2, R28.1, U4.6 (FB)
- new net: D3.2 (K), D6.2 (K), L4.1
- new net: C53.2, R25.1
- new net 1: BT1.1 (+), C56.2, C57.2, R13.2, R28.2, U4.7 (BAT)
- new net CSP: L4.2, R13.1, U4.8 (CSP)
- new net DRAIN: Q1.5 (D), Q1.6 (D), Q1.7 (D), Q1.8 (D)
- new net SOURSE: Q1.1 (S), Q1.2 (S), Q1.3 (S)

Commit message: update of charging and logic
Parts:
- removed C39: 100nf, Capacitor_SMD:C_0805_2012Metric_Pad1.18x1.45mm_HandSolder, symbol Device:C
- added C39: RVT1V101M0607, EasyEDA:CAP-SMD_BD6.3-L6.6-W6.6-LS7.6-FD, symbol EasyEDA:RVT1V101M0607
- added D7, D8: SS54_C22452, EasyEDA:SMA_L4.4-W2.8-LS5.4-R-RD, symbol EasyEDA:SS54_C22452
- added LED18: YLED0805G, EasyEDA:LED0805-FD-GREEN, symbol EasyEDA:YLED0805G
- added R26: 10k, PCM_Resistor_SMD_AKL:R_0805_2012Metric_Pad1.20x1.40mm_HandSolder, symbol Device:R
- added R30: 100K, PCM_Resistor_SMD_AKL:R_0805_2012Metric_Pad1.20x1.40mm_HandSolder, symbol Device:R
- added R31: 2.2k, Resistor_SMD:R_0805_2012Metric_Pad1.20x1.40mm_HandSolder, symbol Device:R
- C55: value 1uF -> 0.1uf
Connections:
- net V3_1 is gone; now on net 3.3V: U15.4 (V3)
- net 1: now also D8.1 (A)
- net DRAIN: now also D6.1 (A)
- net GND: now also C39.2, R26.1; no longer C57.1
- net SOURSE: now also C26.2, C54.2, C55.2, D1.1, D4.2, R22.1, R23.1, R24.1, U4.9 (VCC), USB1.A4B9 (VBUS), USB1.B4A9 (VBUS), C39.1, D7.1 (A), R30.2, R31.1
- net SYS: no longer C18.1, C19.1, U7.1 (Vin)
- net CHARG: now reaches U4.3 (nCHRG)
- net CHARG: now also LED18.2 (K)
- net at U4.4 (MPPT): now also R26.2, R30.1
- removed net V5_1: C54.2, C55.2, D1.1, D4.2, D6.1 (A), R22.1, R23.1, R24.1, U4.9 (VCC), USB1.A4B9 (VBUS), USB1.B4A9 (VBUS)
- new net: LED18.1 (A), R31.2
- new net VCC_REG: C18.1, C19.1, D7.2 (K), D8.2 (K), U7.1 (Vin)
Other:
- note added: "DRIVER cargador."
- note added: "Regulador 15V/3.3V"
- note added: "arreglo de diodos para alimentar circuito."
- note removed: "Regulador 12V/3.3V"
- moved on the sheet: BT1, C14, C15, C21, C26, C53, C54, C55, C56, D3, D6, L4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
