File: HARDWARE/HydroScan_V1.kicad_sch (KiCad schematic)
At the start: 163 parts, among them CN2 DB128V-5.08-2P-GN-S, J1 BATERY, Q1 AO4435_C2944310, Q13 2n3904S-RTK/PS_C18536, Q14 2n3904S-RTK/PS_C18536, Q15 2n3904S-RTK/PS_C18536, Q16 2n3904S-RTK/PS_C18536, SW2 BOOT, SW4 RESET, U1 IP2312-4V35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

Commit message: power updating
Parts:
- removed C20, C32: 0.1uf, Capacitor_SMD:C_0201_0603Metric, symbol Device:C
- removed C25: 4.7uf, PCM_Capacitor_SMD_AKL:C_0805_2012Metric_Pad1.18x1.45mm_HandSolder, symbol Device:C
- removed C27, C28, C36: 47nf, PCM_Capacitor_SMD_AKL:C_0805_2012Metric_Pad1.18x1.45mm_HandSolder, symbol Device:C
- removed C29, C30, C31, C41, C42, C46, C47, C49, C50: 10uf, PCM_Capacitor_SMD_AKL:C_0805_2012Metric_Pad1.18x1.45mm_HandSolder, symbol Device:C
- removed C33, C34, C35: 25TQC33MYF, EasyEDA:CAP-SMD_L7.3-W4.3-FD, symbol EasyEDA:25TQC33MYF
- removed C43, C48: 0.1uf, PCM_Capacitor_SMD_AKL:C_0805_2012Metric_Pad1.18x1.45mm_HandSolder, symbol Device:C
- removed C44: 22uf, PCM_Capacitor_SMD_AKL:C_0805_2012Metric_Pad1.18x1.45mm_HandSolder, symbol Device:C
- removed C45: 47uf, PCM_Capacitor_SMD_AKL:C_0805_2012Metric_Pad1.18x1.45mm_HandSolder, symbol Device:C
- removed C51, C52: CL32B106KBJNNNE, EasyEDA:C1210, symbol EasyEDA:CL32B106KBJNNNE
- removed C57: 1uF, Capacitor_SMD:C_0805_2012Metric_Pad1.18x1.45mm_HandSolder, symbol Device:C
- removed CN2: DB128V-5.08-2P-GN-S, EasyEDA:CONN-TH_2P-P5.08_DIBO_DB128V-5.08, symbol EasyEDA:DB128V-5.08-2P-GN-S
- removed JP1, JP2, JP3, JP4, JP5: SolderJumper_2_Open, Jumper:SolderJumper-2_P1.3mm_Open_RoundedPad1.0x1.5mm, symbol Jumper:SolderJumper_2_Open
- removed L3: 0420CDMCCDS-1R0MC, EasyEDA:IND-SMD_L4.2-W4.2_MCW-0420, symbol EasyEDA:0420CDMCCDS-1R0MC
- removed LED14: YLED0805G, EasyEDA:LED0805-FD-GREEN, symbol EasyEDA:YLED0805G
- removed R16: 2.2k, Resistor_SMD:R_0805_2012Metric_Pad1.20x1.40mm_HandSolder, symbol Device:R
- removed R19, R20: 10k, PCM_Resistor_SMD_AKL:R_0805_2012Metric_Pad1.20x1.40mm_HandSolder, symbol Device:R
- removed R21: 100, Resistor_SMD:R_0805_2012Metric_Pad1.20x1.40mm_HandSolder, symbol Device:R
- removed R86: 100k, PCM_Resistor_SMD_AKL:R_0805_2012Metric_Pad1.20x1.40mm_HandSolder, symbol Device:R
- removed R87: 127k, PCM_Resistor_SMD_AKL:R_0805_2012Metric_Pad1.20x1.40mm_HandSolder, symbol Device:R
- removed R88: 6.04k, PCM_Resistor_SMD_AKL:R_0805_2012Metric_Pad1.20x1.40mm_HandSolder, symbol Device:R
- removed R89: 5.24k, PCM_Resistor_SMD_AKL:R_0805_2012Metric_Pad1.20x1.40mm_HandSolder, symbol Device:R
- removed R90: 30.31k, PCM_Resistor_SMD_AKL:R_0805_2012Metric_Pad1.20x1.40mm_HandSolder, symbol Device:R
- added C20: CA45-D035K226T, EasyEDA:CAP-SMD_L7.3-W4.3-R-RD, symbol EasyEDA:CA45-D035K226T
- added H1: MountingHole_Pad, symbol Mechanical:MountingHole_Pad
- added M_N1: M_N, Connector_PinHeader_2.00mm:PinHeader_1x01_P2.00mm_Vertical, symbol Connector:TestPoint
- added M_P1: TestPoint, Connector_PinHeader_2.00mm:PinHeader_1x01_P2.00mm_Vertical, symbol Connector:TestPoint
- added U10, U11, U8, U9: DB125-3.81-2P-BK-S, EasyEDA:CONN-TH_2P-P3.81_DB125-3.81-2P-BK-S, symbol EasyEDA:DB125-3.81-2P-BK-S
Connections:
- net 1: now also C20.1
- net 3.3V: now also U8.2
- net GND: now also C20.2, H1.1, U10.1, U11.1; no longer U2.10 (ACDRV2), U2.11 (ACDRV1), U2.27 (GND)
- net V_BATTERY__1: now also U11.2
- net at U2.23 (BAT): no longer names the net of U2.23 (BAT)
- net BATP: no longer names the net of U2.18 (BATP)
- net BTST1: no longer names the net of U2.4 (BTST1)
- net BTST2: no longer names the net of U2.19 (BTST2)
- net REGN: no longer names the net of U2.5 (REGN)
- net SDRV: no longer names the net of U2.24 (SDRV)
- net SOURSE renamed V5_1
- net STAT: no longer names the net of U2.1 (STAT)
- net SW1: no longer names the net of U2.28 (SW1)
- net SW2: no longer names the net of U2.26 (SW2)
- net SYS: no longer names the net of U2.25 (SYS)
- net TS: no longer names the net of U2.16 (TS)
- removed net VAC1: U2.2 (VBUS), U2.3 (VBUS), U2.9 (VAC1)
- net VAC2: no longer names the net of U2.8 (VAC2)
- new net: M_N1.1, U8.1
- new net: M_P1.1, U10.2
- no-connect marks 33 -> 31
Other:
- note added: "Asignarle pines a V y A"
- note added: "Motor"
- note removed: "Colocar un conector aqui para el Thermistor NTC"
- note removed: "El ESP32_puede saber en que estado esta la carga y si hay algun problema."
- note removed: "NOTA: C20 AND VBUS pegado posible al pin VBUS LUego los de 10UF"
- note removed: "NOTA: C25 lo mas pegado posible al pin REGN"
- note removed: "NOTA: C27 y todo lo de este cuadro incluyendo inductor pegado al IC RUTEO DE ALTA VELOCIDAD 1.5 MHZ"
- note removed: "NOTA: C29 C31 Y C30 van pegado posible al pin PMID pistas diminutamente cortas mucha corriente"
- note removed: "NOTA: R88 pegado a IC"
- note removed: "NOTA: la menor cantidad de cobre posibles esto irradia mucho ruido por la conmutacion alta, no rutear nada por debajo."
- note removed: "NOTA:Temperatura de bateria detector."
- note removed: "Pin donde se alimentara todo regulador ETC"
- note removed: "conectar a GPIO"

Commit message: powering rooting finish
Parts:
- removed C39: RVT1V101M0607, EasyEDA:CAP-SMD_BD6.3-L6.6-W6.6-LS7.6-FD, symbol EasyEDA:RVT1V101M0607
- removed C54: 10uF, Capacitor_SMD:C_0805_2012Metric_Pad1.18x1.45mm_HandSolder, symbol Device:C
- removed R28: 9110K, PCM_Resistor_SMD_AKL:R_0805_2012Metric_Pad1.20x1.40mm_HandSolder, symbol Device:R
- added C25: RVT1V221M0810, EasyEDA:CAP-SMD_BD8.0-L8.3-W8.3-LS9.1-FD, symbol EasyEDA:RVT1V221M0810
- added C27, C28, C29, C30: CL32B106KBJNNNE, EasyEDA:C1210, symbol EasyEDA:CL32B106KBJNNNE
- added C57: 0.1uf, Capacitor_SMD:C_0805_2012Metric_Pad1.18x1.45mm_HandSolder, symbol Device:C
- added H2: 2.54-2*10, EasyEDA:HDR-TH_20P-P2.54-V-M-R2-C10-S2.54, symbol EasyEDA:2.54-2*10
- added M_N2: M_GND, Connector_PinHeader_2.00mm:PinHeader_1x01_P2.00mm_Vertical, symbol Connector:TestPoint
- added NT1: NetTie_2, NetTie:NetTie-2_SMD_Pad0.5mm, symbol Device:NetTie_2
- added R16: RC0805FR-07390KL, EasyEDA:R0805, symbol EasyEDA:RC0805FR-07390KL
- added VCC_Motor1: M_VCC, Connector_PinHeader_2.00mm:PinHeader_1x01_P2.00mm_Vertical, symbol Connector:TestPoint
- C56: value 10uF -> 0.1uf
- R27: value 100K -> 41.2K; footprint PCM_Resistor_SMD_AKL:R_0805_2012Metric_Pad1.20x1.40mm_HandSolder -> Resistor_SMD:R_0805_2012Metric_Pad1.20x1.40mm_HandSolder; LCSC (none) -> C2077335
Connections:
- net V_BATTERY__1 is gone; now on net VCC_MOTOR: F1.1, U11.2
- net 3.3V: now also H2.1, H2.2
- net GND: now also C25.2, C27.1, C28.1, C29.1, C30.1, C57.1, H2.3, H2.4, M_N2.1, NT1.1; no longer C53.1, R26.1, R27.1, U4.2 (GND)
- net V5_1: now also C25.1, C27.2, C29.2, C57.2
- net VCC_REG: now also C56.2
- net at R27.2, U4.6 (FB): now also R16.2
- net 1 renamed VCC_MOTOR
- net VCC_MOTOR: now also C28.2, C30.2, R16.1, VCC_Motor1.1; no longer C56.2
- net CSP: no longer names the net of L4.2, R13.1, U4.8 (CSP)
- net DRAIN: no longer names the net of D6.1 (A), Q1.5 (D), Q1.6 (D), Q1.7 (D), Q1.8 (D)
- new net GND2: C53.1, NT1.2, R26.1, R27.1, U4.2 (GND)
Other:
- note removed: "DRIVER cargador."
- moved on the sheet: BT1, C20, C26, D7, D8, Q1, U2

Commit message: Update of design the power
update of charging
Parts:
- added C58: 0.1uf, Capacitor_SMD:C_0805_2012Metric_Pad1.18x1.45mm_HandSolder, symbol Device:C
- added INA1: INA, Connector_PinHeader_2.00mm:PinHeader_1x01_P2.00mm_Vertical, symbol Connector:TestPoint
- added INB1: INB, Connector_PinHeader_2.00mm:PinHeader_1x01_P2.00mm_Vertical, symbol Connector:TestPoint
- added PWM1: PWM_1, Connector_PinHeader_2.00mm:PinHeader_1x01_P2.00mm_Vertical, symbol Connector:TestPoint
- added R28, R32, R33, R34: 4.7K, Resistor_SMD:R_0805_2012Metric_Pad1.20x1.40mm_HandSolder, symbol Device:R
Connections:
- net 3.3V: now also H2.19, H2.20, C58.2, R28.2, R32.1, R33.1, R34.1
- net GND: now also C58.1
- net IO17_1: now also H2.12
- net IO21_1: now also H2.15, H2.16, R28.1
- net IO22_1: now also H2.17, H2.18, R32.2
- net IO25_1: now also U9.2, R33.2
- net IO26_1: now also U9.1, R34.2
- net IO27_1: now also H2.11, PWM1.1
- net IO32_1: now also INB1.1
- net IO33_1: now also INA1.1
Other:
- moved on the sheet: C29, C30, C56, C57, D7, D8, M_N2, VCC_Motor1

Commit message: latest updates
Parts:
- removed D2: SS14, PCM_Diode_SMD_AKL:D_SMA, symbol PCM_Diode_Schottky_AKL:SS14
- removed F1: 5x20 BLX-Atype Fuse holder XC-7, EasyEDA:FUSE-TH_L22.6-W9.0, symbol EasyEDA:5x20BLX-AtypeFuseholderXC-7
- removed INA1: INA, Connector_PinHeader_2.00mm:PinHeader_1x01_P2.00mm_Vertical, symbol Connector:TestPoint
- removed LED18: YLED0805G, EasyEDA:LED0805-FD-GREEN, symbol EasyEDA:YLED0805G
- removed U2: BQ25798RQMR, EasyEDA:QFN-29_L4.0-W4.0-P0.40-TL-BQ25792RQMR, symbol EasyEDA:BQ25798RQMR
- added C31: 100nf, Capacitor_SMD:C_0805_2012Metric_Pad1.18x1.45mm_HandSolder, symbol Device:C
- added C59, C60: 0.1uf, Capacitor_SMD:C_0805_2012Metric_Pad1.18x1.45mm_HandSolder, symbol Device:C
- added INB1: INB1, Connector_PinHeader_2.00mm:PinHeader_1x01_P2.00mm_Vertical, symbol Connector:TestPoint
- added R35: 10k, Resistor_SMD:R_0805_2012Metric_Pad1.20x1.40mm_HandSolder, symbol Device:R
- added R36: 30k, Resistor_SMD:R_0805_2012Metric_Pad1.20x1.40mm_HandSolder, symbol Device:R
- added U5: LM358DR, EasyEDA:SOIC-8_L5.0-W4.0-P1.27-LS6.0-BL, symbol EasyEDA:LM358DR
- GND1: renamed from M_N2; value M_GND -> PH_GND
- INB2: renamed from INB1; value INB -> INB2
- PWM1: value PWM_1 -> PWM
- R26, R30, R80: footprint PCM_Resistor_SMD_AKL:R_0805_2012Metric_Pad1.20x1.40mm_HandSolder -> Resistor_SMD:R_0805_2012Metric_Pad1.20x1.40mm_HandSolder
- R31: value 2.2k -> 10k
- renumbered LED12 to 3.3V1, LED15 to BAT1, LED13 to RUN1, LED17 to USB3, VCC_Motor1 to VCC1
Connections:
- net CHARG is gone; now on net IO17_1: U4.3 (nCHRG)
- net 3.3V: now also H2.5, H2.6, R31.2
- net GND: now also H2.10, H2.12, H2.8, C31.1, C59.1, C60.1, R35.1, U5.4 (GND), U5.5 (+IN2)
- net IO13_1: now also H2.18
- net IO14_1: now also INB1.1
- net IO16_1: now also C31.2
- net IO17_1: now also R31.1; no longer H2.12
- net IO18_1: now also H2.11
- net IO19_1: now also RUN1.2 (K)
- net IO21_1: now also H2.13, H2.14; no longer H2.15, H2.16
- net IO22_1: now also H2.15, H2.16; no longer H2.17, H2.18
- net IO23_1: now also H2.17
- net IO25_1: now also R34.2, U9.1; no longer R33.2, U9.2
- net IO26_1: now also PWM1.1; no longer R34.2, U9.1
- net IO27_1: now also INB2.1; no longer H2.11, PWM1.1
- net IO32_1: now also H2.7; no longer INB2.1
- net IO33_1: now also R33.2, U9.2
- net V5_1: no longer R31.1
- net VCC_MOTOR: now also R17.1, R36.2, U5.8 (+V)
- net VN_1: now also C60.2, U5.1 (OUT1), U5.2 (-IN1)
- net VP_1: now also H2.9, C59.2
- net IO12_1: no longer names the net of U16.14 (IO12)
- net IO15_1: no longer names the net of U16.23 (IO15)
- net IO2_1: no longer names the net of U16.24 (IO2)
- net IO4_1: no longer names the net of U16.26 (IO4)
- new net: R35.2, R36.1, U5.3 (+IN1)
- new net: U5.6 (-IN2), U5.7 (OUT2)
- no-connect marks 31 -> 35
Other:
- note added: "Arreglo de diodos para alimentar circuito. Efecto OR"
- note added: "Bateria indicator"
- note added: "CARGADOR_BAT 12.6V"
- note added: "Conector de motor"
- note added: "IO en pines"
- note added: "Linea GND puente H"
- note added: "Linea VCC puente H"
- note added: "PUENTE H INA"
- note added: "PUENTE H INB"
- note added: "PWM del MOTOR"
- note added: "Periferia"
- note added: "Puente_H"
- note added: "Sensor nivel de bateria"
- note added: "Tierra limpia, para medicion exacta."
- note removed: "Asignarle pines a V y A"
- note removed: "CARGADOR_BAT 14.2V"
- note removed: "COMPLICADO"
- note removed: "Pantalla info"
- note removed: "Periferia Botones"
- note removed: "arreglo de diodos para alimentar circuito."
- moved on the sheet: 3.3V1, BAT1, BT1, C20, C25, C26, C27, C28, C29, C30, C53, C55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
