File: HARDWARE/HydroScan_V1.kicad_sch (KiCad schematic)
At the start: 147 parts, among them J1 BATERY, Q1 AO4435_C2944310, Q13 2n3904S-RTK/PS_C18536, Q14 2n3904S-RTK/PS_C18536, Q15 2n3904S-RTK/PS_C18536, Q16 2n3904S-RTK/PS_C18536, SW2 BOOT, SW4 RESET, U1 IP2312-4V35, U10 DB125-3.81-2P-BK-S, U11 DB125-3.81-2P-BK-S, U13 ESP32-WROOM-32D, U14 CH340C, U15 CH340C, U16 ESP32-WROOM-32D, U3 CH224K, U4 CN3795, U5 LM358DR, U7 LM2576HVS-3.3, U8 DB125-3.81-2P-BK-S, U9 DB125-3.81-2P-BK-S

Commit message: correction of errors DRC
Parts:
- removed BOOT1: BOOT, EasyEDA:SW-SMD_4P-L6.0-W6.0-P4.50-LS8.2, symbol EasyEDA:TC-6601-5.0-260-8.3
- removed BT1: Battery, symbol Device:Battery
- removed C1, C4, C6: 10uf_25v, Capacitor_SMD:C_0805_2012Metric_Pad1.18x1.45mm_HandSolder, symbol Device:C
- removed C10, C12, C13: 22uf, Capacitor_SMD:C_0805_2012Metric_Pad1.18x1.45mm_HandSolder, symbol Device:C_Small_US
- removed C11, C9: 10uf, Capacitor_SMD:C_0805_2012Metric_Pad1.18x1.45mm_HandSolder, symbol Device:C_Small_US
- removed C2, C3: 0.1uf_50v, Capacitor_SMD:C_0805_2012Metric_Pad1.18x1.45mm_HandSolder, symbol Device:C
- removed C37, C38: 100nf, PCM_Capacitor_SMD_AKL:C_0805_2012Metric_Pad1.18x1.45mm_HandSolder, symbol Device:C
- removed C5: 100nf, Capacitor_SMD:C_0805_2012Metric_Pad1.18x1.45mm_HandSolder, symbol Device:C
- removed C7, C8: 0.1uf, Capacitor_SMD:C_0805_2012Metric_Pad1.18x1.45mm_HandSolder, symbol Device:C
- removed D22: 1N5819HW-7-F, EasyEDA:SOD-123_L2.7-W1.6-LS3.7-RD, symbol EasyEDA:1N5819HW-7-F
- removed D27, D28, D29, D30, D31: LESD5D5.0CT1G, EasyEDA:SOD-523_L1.2-W0.8-LS1.6-BI, symbol EasyEDA:LESD5D5.0CT1G
- removed H1: MountingHole_Pad, symbol Mechanical:MountingHole_Pad
- removed J1: BATERY, symbol Connector:Conn_01x02_Socket
- removed L1: APH0420T1R0M, EasyEDA:IND-SMD_L4.4-W4.2, symbol EasyEDA:APH0420T1R0M
- removed LED10, LED11, LED16, LED9: YLED0805G, EasyEDA:LED0805-FD-GREEN, symbol EasyEDA:YLED0805G
- removed PH_sensor1: PH-4502C, symbol Mis_creaciones:PH-4502C
- removed Q13, Q15: 2n3904S-RTK/PS_C18536, EasyEDA:SOT-23-3_L2.9-W1.3-P1.90-LS2.4-TR, symbol EasyEDA:2n3904S-RTK_PS_C18536
- removed R1: 2R, Resistor_SMD:R_0805_2012Metric_Pad1.20x1.40mm_HandSolder, symbol Device:R_Small_US
- removed R10: 0.5R, Resistor_SMD:R_0805_2012Metric_Pad1.20x1.40mm_HandSolder, symbol Device:R_Small_US
- removed R18, R6: 2.2k, Resistor_SMD:R_0805_2012Metric_Pad1.20x1.40mm_HandSolder, symbol Device:R
- removed R2: 51k, Resistor_SMD:R_0805_2012Metric_Pad1.20x1.40mm_HandSolder, symbol Device:R_Small_US
- removed R3, R4: 100, Resistor_SMD:R_0805_2012Metric_Pad1.20x1.40mm_HandSolder, symbol Device:R_Small_US
- removed R5, R78: 5.11k, PCM_Resistor_SMD_AKL:R_0805_2012Metric_Pad1.20x1.40mm_HandSolder, symbol Device:R
- removed R7, R8: 10k, PCM_Resistor_SMD_AKL:R_0805_2012Metric_Pad1.20x1.40mm_HandSolder, symbol Device:R
- removed R74, R75: 1k, Resistor_SMD:R_0805_2012Metric_Pad1.20x1.40mm_HandSolder, symbol Device:R
- removed R76, R77: 0, PCM_Resistor_SMD_AKL:R_0805_2012Metric_Pad1.20x1.40mm_HandSolder, symbol Device:R
- removed R9: 1k, Resistor_SMD:R_0805_2012Metric_Pad1.20x1.40mm_HandSolder, symbol Device:R_Small_US
- removed RESET1: RESET, EasyEDA:SW-SMD_4P-L6.0-W6.0-P4.50-LS8.2, symbol EasyEDA:TC-6601-5.0-260-8.3
- removed SGM2212-3.1: (no value), Package_TO_SOT_SMD:SOT-223, symbol PCM_Voltage_Regulator_AKL:SGM2212-3.3XKC3G
- removed U1: IP2312-4V35, EasyEDA:ESOP-8_L4.9-W3.9-P1.27-LS6.0-BL-EP, symbol EasyEDA:IP2312-4V35
- removed U13: ESP32-WROOM-32D, RF_Module:ESP32-WROOM-32D, symbol RF_Module:ESP32-WROOM-32D
- removed U14: CH340C, Package_SO:SOIC-16_3.9x9.9mm_P1.27mm, symbol Interface_USB:CH340C
- removed USB2: HX-TYPE-C 16P 180 LT H15.0, EasyEDA:USB-C-SMD_HX-TYPE-C-16P-180-LT-H15.0, symbol EasyEDA:HX-TYPE-C16P180LTH15.0
Connections:
- no-connect marks 35 -> 21
Other:
- note removed: "CARGADOR_BAT 4.2V"
- note removed: "Indicador de USB 3V"
- note removed: "NOTA: Estos capacitores C37 y C38 deben ir juntos y pegados lo mas que se pueda fisicamente a el IC UART."
- note removed: "NOTA: TX Y RX Va al revez, pero revisa como el ruteado se te hace mas facil TX y RX"
- note removed: "Nota: Estos capacitores C9 y c10 deben ir juntos y pegados lo mas que se pueda fisicamente a el IC."
- note removed: "listo"
- moved on the sheet: C20, C28

Commit message: Update of power desing
Parts:
- R24: footprint Resistor_SMD:R_0805_2012Metric_Pad1.20x1.40mm_HandSolder -> Capacitor_SMD:C_0805_2012Metric_Pad1.18x1.45mm_HandSolder
Other:
- moved on the sheet: C31, R24
Changed lines of the file:
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@@
 	(rectangle
 		(start 434.34 63.5)
-		(end 826.77 196.85)
+		(end 826.77 198.12)
 		(stroke
 			(width 0.0762)
@@
 	(rectangle
 		(start 434.34 49.53)
-		(end 826.77 196.85)
+		(end 826.77 198.12)
 		(stroke
 			(width 0.0762)
@@
 	(rectangle
 		(start 486.41 154.94)
-		(end 612.14 196.85)
+		(end 612.14 198.12)
 		(stroke
 			(width 0)
@@
 	)
 	(rectangle
-		(start 610.87 198.12)
+		(start 612.14 198.12)
 		(end 828.04 215.9)
 		(stroke
@@
 	(text "proteccion TVS\n"
 		(exclude_from_sim no)
-		(at 511.302 125.73 0)
+		(at 511.048 123.19 0)
 		(effects
 			(font
@@
 	)
 	(junction
+		(at 656.59 93.98)
+		(diameter 0)
+		(color 0 0 0 0)
+	)
+	(junction
 		(at 523.24 115.57)
 		(diameter 0)
@@
 	)
 	(junction
-		(at 656.59 93.98)
-		(diameter 0)
-		(color 0 0 0 0)
-	)
-	(junction
 		(at 678.18 102.87)
 		(diameter 0)
@@
 	(wire
 		(pts
-			(xy 556.26 106.68) (xy 552.45 106.68)
-		)
-		(stroke
-			(width 0)
-			(type default)
-		)
-	)
-	(wire
-		(pts
 			(xy 758.19 95.25) (xy 763.27 95.25)
 		)
@@
 	(wire
 		(pts
-			(xy 552.45 111.76) (xy 554.99 111.76)
+			(xy 549.91 110.49) (xy 554.99 110.49)
 		)
 		(stroke
@@
 		)
 	)
+	(wire
+		(pts
+			(xy 631.19 95.25) (xy 631.19 93.98)
+		)
+		(stroke
+			(width 0)
+			(type default)
+		)
+	)
 	(polyline
 		(pts
@@
 	(wire
 		(pts
+			(xy 660.4 93.98) (xy 656.59 93.98)
+		)
+		(stroke
+			(width 0)
+			(type default)
+		)
+	)
+	(wire
+		(pts
 			(xy 681.99 347.98) (xy 690.88 347.98)
 		)
@@
 	(polyline
 		(pts
-			(xy 803.91 93.98) (xy 811.53 93.98)
+			(xy 803.91 90.17) (xy 811.53 90.17)
 		)
 		(stroke
@@
 	(wire
 		(pts
+			(xy 599.44 107.95) (xy 599.44 105.41)
+		)
+		(stroke
+			(width 0)
+			(type default)
+		)
+	)
+	(wire
+		(pts
 			(xy 459.74 106.68) (xy 459.74 105.41)
 		)
@@
 	(wire
 		(pts
+			(xy 562.61 110.49) (xy 562.61 111.76)
+		)
+		(stroke
+			(width 0)
+			(type default)
+		)
+	)
+	(wire
+		(pts
 			(xy 711.2 234.95) (xy 715.01 234.95)
 		)
@@
 	(wire
 		(pts
-			(xy 656.59 97.79) (xy 656.59 93.98)
-		)
-		(stroke
-			(width 0)
-			(type default)
-		)
-	)
-	(wire
-		(pts
 			(xy 523.24 109.22) (xy 523.24 115.57)
 		)
@@
 	(wire
 		(pts
-			(xy 552.45 106.68) (xy 552.45 111.76)
-		)
-		(stroke
-			(width 0)
-			(type default)
-		)
-	)
-	(wire
-		(pts
 			(xy 599.44 105.41) (xy 608.33 105.41)
 		)
@@
 	(wire
 		(pts
+			(xy 656.59 93.98) (xy 656.59 97.79)
+		)
+		(stroke
+			(width 0)
+			(type default)
+		)
+	)
+	(wire
+		(pts
 			(xy 759.46 326.39) (xy 759.46 328.93)
 		)
@@
 	(wire
 		(pts
+			(xy 599.44 118.11) (xy 599.44 115.57)
+		)
+		(stroke
+			(width 0)
+			(type default)
+		)
+	)
+	(wire
+		(pts
 			(xy 687.07 260.35) (xy 687.07 267.97)
 		)
@@
 	(wire
 		(pts
-			(xy 631.19 93.98) (xy 631.19 95.25)
-		)
-		(stroke
-			(width 0)
-			(type default)
-		)
-	)
-	(wire
-		(pts
 			(xy 650.24 267.97) (xy 657.86 267.97)
 		)
@@
 	(polyline
 		(pts
-			(xy 803.91 88.9) (xy 811.53 88.9)
+			(xy 803.91 87.63) (xy 811.53 87.63)
 		)
 		(stroke
@@
 	(polyline
 		(pts
-			(xy 802.64 106.68) (xy 811.53 106.68)
+			(xy 803.91 95.25) (xy 811.53 95.25)
 		)
 		(stroke
@@
 	(wire
 		(pts
-			(xy 656.59 88.9) (xy 656.59 93.98)
-		)
-		(stroke
-			(width 0)
-			(type default)
-		)
-	)
-	(wire
-		(pts
 			(xy 499.11 143.51) (xy 499.11 142.24)
 		)
@@
 	)
 	(label "EN"
-		(at 656.59 88.9 270)
+		(at 660.4 93.98 180)
 		(effects
 			(font
@@
 	)
 	(label "V5_1"
-		(at 556.26 106.68 180)
+		(at 549.91 110.49 0)
 		(effects
 			(font
 				(size 1.27 1.27)
 			)
-			(justify right bottom)
+			(justify left bottom)
 		)
 	)
@@
 	(symbol
 		(lib_id "power:+5V")
-		(at 599.44 96.52 270)
+		(at 599.44 96.52 0)
 		(unit 1)
 		(body_style 1)
@@
 		(dnp no)
 		(property "Reference" "#PWR038"
-			(at 595.63 96.52 0)
+			(at 599.44 100.33 0)
 			(hide yes)
 			(show_name no)
@@
 		)
 		(property "Value" "3.3V"
-			(at 601.98 96.774 90)
+			(at 598.17 92.964 0)
 			(show_name no)
 			(do_not_autoplace no)
@@
 	(symbol
 		(lib_id "Device:R")
-		(at 558.8 111.76 90)
+		(at 558.8 110.49 90)
 		(mirror x)
 		(unit 1)
@@
 		(dnp no)
 		(property "Reference" "R24"
-			(at 560.578 111.76 90)
+			(at 560.578 110.49 90)
 			(show_name no)
 			(do_not_autoplace no)
@@
 		)
 		(property "Value" "10k"
-			(at 556.768 109.982 90)
+			(at 556.768 108.712 90)
 			(show_name no)
 			(do_not_autoplace no)
@@
 			)
 		)
-		(property "Footprint" "Resistor_SMD:R_0805_2012Metric_Pad1.20x1.40mm_HandSolder"
-			(at 558.8 109.982 90)
+		(property "Footprint" "Capacitor_SMD:C_0805_2012Metric_Pad1.18x1.45mm_HandSolder"
+			(at 558.8 108.712 90)
 			(hide yes)
 			(show_name no)
@@
 		)
 		(property "Datasheet" ""
-			(at 558.8 111.76 0)
+			(at 558.8 110.49 0)
 			(hide yes)
 			(show_name no)
@@
 		)
 		(property "Description" "Resistor"
-			(at 558.8 111.76 0)
+			(at 558.8 110.49 0)
 			(hide yes)
 			(show_name no)
@@
 	(symbol
 		(lib_id "power:GND")
-		(at 599.44 113.03 0)
+		(at 599.44 118.11 0)
 		(mirror y)
 		(unit 1)
@@
 		(dnp no)
 		(property "Reference" "#PWR061"
-			(at 599.44 119.38 0)
+			(at 599.44 124.46 0)
 			(hide yes)
 			(show_name no)
@@
 		)
 		(property "Value" "GND"
-			(at 599.44 116.586 0)
+			(at 599.44 121.666 0)
 			(show_name no)
 			(do_not_autoplace no)
@@
 		)
 		(property "Footprint" ""
-			(at 599.44 113.03 0)
+			(at 599.44 118.11 0)
 			(hide yes)
 			(show_name no)
@@
 		)
 		(property "Datasheet" ""
-			(at 599.44 113.03 0)
+			(at 599.44 118.11 0)
 			(hide yes)
 			(show_name no)
@@
 		)
 		(property "Description" "Power symbol creates a global label with name \"GND\" , ground"
-			(at 599.44 113.03 0)
+			(at 599.44 118.11 0)
 			(hide yes)
 			(show_name no)
@@
 	(symbol
 		(lib_id "Device:C")
-		(at 599.44 109.22 180)
+		(at 599.44 111.76 180)
 		(unit 1)
 		(body_style 1)
@@
 		(dnp no)
 		(property "Reference" "C31"
-			(at 601.218 109.22 0)
+			(at 601.218 111.76 0)
 			(show_name no)
 			(do_not_autoplace no)
@@
 		)
 		(property "Value" "100nf"
-			(at 599.44 107.188 0)
+			(at 599.44 109.728 0)
 			(show_name no)
 			(do_not_autoplace no)
@@
 		)
 		(property "Footprint" "Capacitor_SMD:C_0805_2012Metric_Pad1.18x1.45mm_HandSolder"
-			(at 598.4748 105.41 0)
+			(at 598.4748 107.95 0)
 			(hide yes)
 			(show_name no)
@@
 		)
 		(property "Datasheet" ""
-			(at 599.44 109.22 0)
+			(at 599.44 111.76 0)
 			(hide yes)
 			(show_name no)
@@
 		)
 		(property "Description" "Unpolarized capacitor"
-			(at 599.44 109.22 0)
+			(at 599.44 111.76 0)
 			(hide yes)
 			(show_name no)

Commit message: squematic update of USB 15V
Other:
- note added: "Proteccion TVS"
- note removed: "proteccion TVS"
- moved on the sheet: C22, C23, C31, D1, D4, R23, R24, R29, R84, R85, U11, USB1

Commit message: update of desing Ambu and hydro
Parts:
- added H1, H3: HX PZ2.54-1X16P ZZ, EasyEDA:HDR-TH_16P-P2.54-V-M_2, symbol EasyEDA:HXPZ2.54-1X16PZZ
- added H4: PZ254V-11-04P_C2691448, EasyEDA:HDR-TH_4P-P2.54-V-M, symbol EasyEDA:PZ254V-11-04P_C2691448
Connections:
- net GND: now also H1.13, H1.14, H1.15, H1.2, H3.12, H3.15, H3.4
- new net 3.3V+: H1.1, H3.3
- new net IO0: H3.13
- new net IO1: H3.5
- new net IO10: H1.7
- new net IO11: H1.8
- new net IO12: H1.9
- new net IO2: H3.6
- new net IO3: H1.4
- new net IO38: H3.11
- new net IO39: H3.10
- new net IO40: H3.9
- new net IO41: H3.8
- new net IO42: H3.7
- new net IO45: H1.11
- new net IO46: H1.5
- new net IO48: H1.12
- new net IO5: H1.3
- new net IO8: H1.10
- new net IO9: H1.6
- new net RST: H3.14
- new net UART0_RX: H3.2
- new net UART0_TX: H3.1
- new net VBUS: H3.16
- new net V_BAT: H1.16
Other:
- note added: "Conectores"
- note added: "MODULO"
- note added: "STEP UP"
- note removed: "Nota problemas: /Comunicacion /Alimentacion /bateria"
- note removed: "PERIFERIA_ILUMINARIA"
- note removed: "Regulador 3V"
- note removed: "SENSOR_PH"
- note removed: "SENSOR_VIA_SONDA_IDC"
