File: HARDWARE/HydroScan_V1.kicad_sch (KiCad schematic)
At the start: 95 parts, among them Q1 AO4435_C2944310, Q14 2n3904S-RTK/PS_C18536, Q16 2n3904S-RTK/PS_C18536, SW2 BOOT, SW4 RESET, U10 DB125-3.81-2P-BK-S, U11 DB125-3.81-2P-BK-S, U15 CH340C, U16 ESP32-WROOM-32D, U3 CH224K, U4 CN3795, U5 LM358DR, U7 LM2576HVS-3.3, U8 DB125-3.81-2P-BK-S, U9 DB125-3.81-2P-BK-S

Commit message: DRC update
Parts:
- added 3.3V2: 3V, TestPoint:TestPoint_Pad_2.5x2.5mm, symbol Connector:TestPoint
- added 5V1: 5V, TestPoint:TestPoint_Pad_2.5x2.5mm, symbol Connector:TestPoint
- added C32, C33, C34: 10uf_25v, Capacitor_SMD:C_0805_2012Metric_Pad1.18x1.45mm_HandSolder, symbol Device:C
- added C61, C62, C63: 0.1uf, Capacitor_SMD:C_0805_2012Metric_Pad1.18x1.45mm_HandSolder, symbol Device:C
- added DC1: DC-470-2.1GP, EasyEDA:DC-IN-TH_DC-470-2.1GP, symbol EasyEDA:DC-470-2.1GP
- added GND2: GND, TestPoint:TestPoint_Pad_2.5x2.5mm, symbol Connector:TestPoint
- added H5: 2.54-2*10, EasyEDA:HDR-TH_20P-P2.54-V-M-R2-C10-S2.54, symbol EasyEDA:2.54-2*10
- added J1: Conn_01x08_Pin, EasyEDA:MPU6050_Module, symbol Connector:Conn_01x08_Pin
- added J2: Conn_01x03_Pin, Connector_PinHeader_2.54mm:PinHeader_1x03_P2.54mm_Vertical, symbol Connector:Conn_01x03_Pin
- added JP1: SolderJumper_3_Open, Jumper:SolderJumper-3_P1.3mm_Open_RoundedPad1.0x1.5mm_NumberLabels, symbol Jumper:SolderJumper_3_Open
- added JP2: SolderJumper_2_Open, Jumper:SolderJumper-2_P1.3mm_Open_Pad1.0x1.5mm, symbol Jumper:SolderJumper_2_Open
- added R37, R38: 4.7K, Resistor_SMD:R_0805_2012Metric_Pad1.20x1.40mm_HandSolder, symbol Device:R
- added R40: 6.8k, Resistor_SMD:R_0805_2012Metric_Pad1.20x1.40mm_HandSolder, symbol Device:R
- added U1: SY6280AAC, EasyEDA:SOT-23-5_L3.0-W1.7-P0.95-LS2.8-BL, symbol EasyEDA:SY6280AAC
Connections:
- net 3.3V+: now also H4.1, 3.3V2.1, C32.1, C62.2, H5.11, H5.12, J1.8 (Pin_8), JP1.1 (A), R37.2, R38.2
- net GND: now also H4.2, H4.3, C32.2, C33.2, C34.2, C61.1, C62.1, C63.1, DC1.2, DC1.3, GND2.1, H5.17, H5.18, H5.19, H5.20, H5.4, H5.5, J1.2 (Pin_2), J1.7 (Pin_7), J2.1 (Pin_1), R40.1, U1.2 (GND)
- net IO1: now also H5.7
- net IO10: now also H5.3
- net IO11: now also H5.6
- net IO12: now also H5.8
- net IO2: now also J2.3 (Pin_3)
- net IO5: now also U1.4 (EN)
- net IO8: now also H5.2, J1.6 (Pin_6), R38.1
- net IO9: now also H5.1, J1.5 (Pin_5), R37.1
- net V5_1: now also DC1.1
- net OUT_PUT_ UP: now reaches H4.4
- net OUT_PUT_ UP: now also C33.1, C34.1, C61.2, U1.5 (IN)
- net IO38 renamed INT
- net INT: now also J1.1 (Pin_1)
- net V_BAT renamed BAT_2_1
- net BAT_2_1: now also JP2.1 (A)
- new net: R40.2, U1.3 (ISET)
- new net: J2.2 (Pin_2), JP1.2 (C)
- new net +5V: 5V1.1, C63.2, H5.15, H5.16, JP1.3 (B), U1.1 (OUT)
- new net BAT_2: JP2.2 (B)
- new net XCL: J1.3 (Pin_3)
- new net XDA: J1.4 (Pin_4)
- no-connect marks 21 -> 29
Other:
- note added: "GYRO"
- note added: "I2C"
- note added: "SCL"
- note added: "SDA"
- note added: "Temp"
- note added: "pines del esp32 INT IO38 para muestras por espera SDA IO9 SCL IO8"
- moved on the sheet: 3.3V1, BAT1, C20, C24, C25, C26, C27, C28, C29, C30, C53, C55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

Commit message: PCB_v1
manufacturing list
Parts:
- added 3.3V3, BATTERY1, GND3, USB2: TestPoint, TestPoint:TestPoint_Pad_2.0x2.0mm, symbol Connector:TestPoint
- added C64: 0.1uf, Capacitor_SMD:C_0805_2012Metric_Pad1.18x1.45mm_HandSolder, symbol Device:C
- added JP3: SolderJumper_3_Open, Jumper:SolderJumper-3_P1.3mm_Open_RoundedPad1.0x1.5mm_NumberLabels, symbol Jumper:SolderJumper_3_Open
- added JP4, JP5: SolderJumper_2_Open, Jumper:SolderJumper-2_P1.3mm_Open_Pad1.0x1.5mm, symbol Jumper:SolderJumper_2_Open
- added R39, R41: 100K, Resistor_SMD:R_0805_2012Metric_Pad1.20x1.40mm_HandSolder, symbol Device:R
- 3.3V1, BAT1, RUN1, USB3: MPN (none) -> YLED0805G; Manufacturer (none) -> YONGYUTAI(永裕泰)
- renumbered H4 to DC_BOOST_1, H1 to H5.1, H3 to H5.2
Connections:
- net +5V: now also C33.1, C61.2, DC_BOOST_1.4, JP3.3 (B); no longer C63.2, U1.1 (OUT)
- net 3.3V: now also 3.3V3.1
- net 3.3V+: now also C34.1, U1.5 (IN), JP4.1 (A), JP5.2 (B); no longer C32.1, C62.2, DC_BOOST_1.1, J1.8 (Pin_8), JP1.1 (A)
- net BAT_2: now also R41.2
- net GND: now also C64.1, GND3.1, R39.1
- net IO1: now also C64.2, R39.2, R41.1; no longer H5.7
- net IO48: now also H5.10
- net UART0_RX: now also H5.9
- net UART0_TX: now also H5.7
- net V5_1: now also JP5.1 (A), USB2.1
- net 3.3V+_1: now reaches H5.13
- net 3.3V+_1: now also C32.1, C62.2, C63.2, DC_BOOST_1.1, H5.14, JP1.1 (A), U1.1 (OUT), JP3.1 (A), JP4.2 (B)
- net IO34_1: no longer names the net of U16.6 (IO34)
- net IO35_1: no longer names the net of U16.7 (IO35)
- net IO5_1: no longer names the net of U16.29 (IO5)
- removed net OUT_PUT_ UP: C33.1, C34.1, C61.2, DC_BOOST_1.4, U1.5 (IN)
- net VCC_MOTOR renamed V_BATTERY__1
- net V_BATTERY__1: now also BATTERY1.1
- new net: J1.8 (Pin_8), JP3.2 (C)
- no-connect marks 29 -> 36
Other:
- note added: "BAT sensor"
- note added: "En caso de que se quiera siempre encendidos los sensores"
- note added: "Este solo es para la producccion nunca unir aunque se va a romper cuando cortemos"
- note added: "GYROSCOPE"
- note added: "Jumper de pin de batteria del modulo, no es la entrada del voltaje principal"
- note added: "Medidor de bateria"
- note added: "NOTA: Pines del ESP32 para muestras por espera (INT IO38) Datos: SDA IO9 SCL IO8"
- note added: "Nota: Esto es para elegir a que voltaje operara y tambien conmutara la carga."
- note added: "Puntos de prueba"
- note added: "TEMP sensor"
- note added: "Tierra 2 limpia, para medicion exacta."
- note added: "nota: no soldar a menos que sea necesario"
- note removed: "GYRO"
- note removed: "Tierra limpia, para medicion exacta."
- note removed: "pines del esp32 INT IO38 para muestras por espera SDA IO9 SCL IO8"
- moved on the sheet: 3.3V2, 5V1, C32, C33, C34, C61, C62, C63, DC_BOOST_1, GND2, H5, H5.1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

Commit message: BOM generate
Parts:
- added BATTERY2: TestPoint, TestPoint:TestPoint_Pad_2.0x2.0mm, symbol Connector:TestPoint
- added JP6, JP7: SolderJumper_3_Open, Jumper:SolderJumper-3_P1.3mm_Open_RoundedPad1.0x1.5mm_NumberLabels, symbol Jumper:SolderJumper_3_Open
- added R1: TC33X-2-103E, EasyEDA:RES-ADJ-SMD_3P-L3.0-W3.8-P1.75-BR, symbol EasyEDA:TC33X-2-103E
- added R42, R43: 10k, Resistor_SMD:R_0805_2012Metric_Pad1.20x1.40mm_HandSolder, symbol Device:R
- added TP1: TDS_1, TestPoint:TestPoint_THTPad_D4.0mm_Drill2.0mm, symbol Connector:TestPoint
- added TP2: TDS_2, TestPoint:TestPoint_THTPad_D4.0mm_Drill2.0mm, symbol Connector:TestPoint
Connections:
- net 3.3V: now also JP6.3 (B), JP7.3 (B)
- net GND: now also JP6.1 (A), JP7.1 (A)
- net IO23_1: now also R42.2
- net IO32_1: now also R43.2
- net V_BATTERY__1: now also BATTERY2.1
- new net: R1.1, TP1.1
- new net: R1.2, TP2.1
- new net: JP6.2 (C), R42.1
- new net: JP7.2 (C), R43.1
- no-connect marks 36 -> 37
Other:
- note added: "TDS potenciometer"
- note removed: "Temp"
- moved on the sheet: H5, J2, JP1, JP4, JP5, R37, R38
