File: HARDWARE/HydroScan_V1.kicad_pcb (KiCad board)
At the start: 4 copper layers, 202 x 100 mm, 101 parts, among them Q1 AO4435_C2944310, Q14 2n3904S-RTK/PS_C18536, Q16 2n3904S-RTK/PS_C18536, SW2 BOOT, SW4 RESET, U10 DB125-3.81-2P-BK-S, U11 DB125-3.81-2P-BK-S, U13 ESP32-WROOM-32D, U15 CH340C, U16 ESP32-WROOM-32D, U2 L298N, U3 CH224K, U4 CN3795, U5 LM358DR, U7 LM2576HVS-3.3, U8 DB125-3.81-2P-BK-S, U9 DB125-3.81-2P-BK-S

Commit message: Hydrofish
update pcb
Parts:
- added BOOT1: BOOT, EasyEDA:SW-SMD_4P-L6.0-W6.0-P4.50-LS8.2, F.Cu at (232.4, 174.7)
- added C1: 10uf_25v, Capacitor_SMD:C_0805_2012Metric_Pad1.18x1.45mm_HandSolder, F.Cu at (214.9, 172.5)
- added C10: 22uf, Capacitor_SMD:C_0805_2012Metric_Pad1.18x1.45mm_HandSolder, F.Cu at (219.7, 184.5)
- added C11: 10uf, Capacitor_SMD:C_0805_2012Metric_Pad1.18x1.45mm_HandSolder, F.Cu at (224.5, 172.5)
- added C12: 22uf, Capacitor_SMD:C_0805_2012Metric_Pad1.18x1.45mm_HandSolder, F.Cu at (224.5, 175.5)
- added C13: 22uf, Capacitor_SMD:C_0805_2012Metric_Pad1.18x1.45mm_HandSolder, F.Cu at (224.5, 178.5)
- added C2: 0.1uf_50v, Capacitor_SMD:C_0805_2012Metric_Pad1.18x1.45mm_HandSolder, F.Cu at (214.9, 175.5)
- added C3: 0.1uf_50v, Capacitor_SMD:C_0805_2012Metric_Pad1.18x1.45mm_HandSolder, F.Cu at (214.9, 178.5)
- added C4: 10uf_25v, Capacitor_SMD:C_0805_2012Metric_Pad1.18x1.45mm_HandSolder, F.Cu at (214.9, 181.5)
- added C5: 100nf, Capacitor_SMD:C_0805_2012Metric_Pad1.18x1.45mm_HandSolder, F.Cu at (214.9, 184.5)
- added C6: 10uf_25v, Capacitor_SMD:C_0805_2012Metric_Pad1.18x1.45mm_HandSolder, F.Cu at (219.7, 172.5)
- added C7: 0.1uf, Capacitor_SMD:C_0805_2012Metric_Pad1.18x1.45mm_HandSolder, F.Cu at (219.7, 175.5)
- added C8: 0.1uf, Capacitor_SMD:C_0805_2012Metric_Pad1.18x1.45mm_HandSolder, F.Cu at (219.7, 178.5)
- added C9: 10uf, Capacitor_SMD:C_0805_2012Metric_Pad1.18x1.45mm_HandSolder, F.Cu at (219.7, 181.5)
- added D22: 1N5819HW-7-F, EasyEDA:SOD-123_L2.7-W1.6-LS3.7-RD, F.Cu at (267.6, 183.2)
- added D27: LESD5D5.0CT1G, EasyEDA:SOD-523_L1.2-W0.8-LS1.6-BI, F.Cu at (266.6, 172.1)
- added D28: LESD5D5.0CT1G, EasyEDA:SOD-523_L1.2-W0.8-LS1.6-BI, F.Cu at (266.6, 174.2)
- added D29: LESD5D5.0CT1G, EasyEDA:SOD-523_L1.2-W0.8-LS1.6-BI, F.Cu at (266.6, 176.3)
- added D30: LESD5D5.0CT1G, EasyEDA:SOD-523_L1.2-W0.8-LS1.6-BI, F.Cu at (266.6, 178.4)
- added D31: LESD5D5.0CT1G, EasyEDA:SOD-523_L1.2-W0.8-LS1.6-BI, F.Cu at (266.6, 180.6)
- added H2: MountingHole_3.2mm_M3_DIN965_Pad_TopBottom, MountingHole:MountingHole_3.2mm_M3_DIN965_Pad_TopBottom, F.Cu at (297.9, 190.4)
- added H2: MountingHole_3.2mm_M3_DIN965_Pad_TopBottom, MountingHole:MountingHole_3.2mm_M3_DIN965_Pad_TopBottom, F.Cu at (186.0, 190.7)
- added H2: MountingHole_3.2mm_M3_DIN965_Pad_TopBottom, MountingHole:MountingHole_3.2mm_M3_DIN965_Pad_TopBottom, F.Cu at (185.9, 147.9)
- added H2: MountingHole_3.2mm_M3_DIN965_Pad_TopBottom, MountingHole:MountingHole_3.2mm_M3_DIN965_Pad_TopBottom, F.Cu at (297.2, 148.6)
- added L1: APH0420T1R0M, EasyEDA:IND-SMD_L4.4-W4.2, F.Cu at (265.2, 165.3)
- added LED10: YLED0805G, EasyEDA:LED0805-FD-GREEN, F.Cu at (253.8, 176.0)
- added LED11: YLED0805G, EasyEDA:LED0805-FD-GREEN, F.Cu at (253.8, 179.3)
- added LED16: YLED0805G, EasyEDA:LED0805-FD-GREEN, F.Cu at (253.8, 182.6)
- added LED9: YLED0805G, EasyEDA:LED0805-FD-GREEN, F.Cu at (253.8, 172.7)
- added Q13: 2n3904S-RTK/PS_C18536, EasyEDA:SOT-23-3_L2.9-W1.3-P1.90-LS2.4-TR, F.Cu at (264.4, 148.2)
- added Q15: 2n3904S-RTK/PS_C18536, EasyEDA:SOT-23-3_L2.9-W1.3-P1.90-LS2.4-TR, F.Cu at (264.4, 152.4)
- added R1: 2R, Resistor_SMD:R_0805_2012Metric_Pad1.20x1.40mm_HandSolder, F.Cu at (279.8, 160.4)
- added R10: 0.5R, Resistor_SMD:R_0805_2012Metric_Pad1.20x1.40mm_HandSolder, F.Cu at (284.5, 160.4)
- added R18: 2.2k, Resistor_SMD:R_0805_2012Metric_Pad1.20x1.40mm_HandSolder, F.Cu at (284.5, 163.3)
- added R2: 51k, Resistor_SMD:R_0805_2012Metric_Pad1.20x1.40mm_HandSolder, F.Cu at (279.8, 163.3)
- added R3: 100, Resistor_SMD:R_0805_2012Metric_Pad1.20x1.40mm_HandSolder, F.Cu at (279.8, 166.3)
- added R4: 100, Resistor_SMD:R_0805_2012Metric_Pad1.20x1.40mm_HandSolder, F.Cu at (279.8, 169.2)
- added R6: 2.2k, Resistor_SMD:R_0805_2012Metric_Pad1.20x1.40mm_HandSolder, F.Cu at (279.8, 172.2)
- added R74: 1k, Resistor_SMD:R_0805_2012Metric_Pad1.20x1.40mm_HandSolder, F.Cu at (284.5, 166.3)
- added R75: 1k, Resistor_SMD:R_0805_2012Metric_Pad1.20x1.40mm_HandSolder, F.Cu at (284.5, 169.2)
- added R9: 1k, Resistor_SMD:R_0805_2012Metric_Pad1.20x1.40mm_HandSolder, F.Cu at (279.8, 175.1)
- added REF**: WEEE-Logo_5.6x8mm_SilkScreen, Symbol:WEEE-Logo_5.6x8mm_SilkScreen, B.Cu at (237.1, 147.8)
- added RESET1: RESET, EasyEDA:SW-SMD_4P-L6.0-W6.0-P4.50-LS8.2, F.Cu at (232.4, 182.0)
- added SGM2212-3.1: ~, Package_TO_SOT_SMD:SOT-223, F.Cu at (242.8, 181.4)
- added THECPCENTER: LOGO, images:IMG1, F.Cu at (241.6, 168.5)
- added U1: IP2312-4V35, EasyEDA:ESOP-8_L4.9-W3.9-P1.27-LS6.0-BL-EP, F.Cu at (265.8, 158.5)
- added U14: CH340C, Package_SO:SOIC-16_3.9x9.9mm_P1.27mm, F.Cu at (260.8, 176.9)
- added USB2: HX-TYPE-C 16P 180 LT H15.0, EasyEDA:USB-C-SMD_HX-TYPE-C-16P-180-LT-H15.0, F.Cu at (244.5, 174.1)
- moved U13 35.9 mm to (237.2, 160.0), turned to 0 degrees
Routing:
- net /IO17_1: track 97.0 -> 98.7 mm
- net /IO33_1: track 81.2 -> 82.4 mm
- net /VN_1: track 40.3 -> 39.4 mm
Other:
- board size 202 x 100 mm -> 222 x 100 mm

Commit message: correction of errors DRC
Parts:
- removed BOOT1: BOOT, EasyEDA:SW-SMD_4P-L6.0-W6.0-P4.50-LS8.2
- removed C1, C4, C6: 10uf_25v, Capacitor_SMD:C_0805_2012Metric_Pad1.18x1.45mm_HandSolder
- removed C10, C12, C13: 22uf, Capacitor_SMD:C_0805_2012Metric_Pad1.18x1.45mm_HandSolder
- removed C11, C9: 10uf, Capacitor_SMD:C_0805_2012Metric_Pad1.18x1.45mm_HandSolder
- removed C2, C3: 0.1uf_50v, Capacitor_SMD:C_0805_2012Metric_Pad1.18x1.45mm_HandSolder
- removed C5: 100nf, Capacitor_SMD:C_0805_2012Metric_Pad1.18x1.45mm_HandSolder
- removed C7, C8: 0.1uf, Capacitor_SMD:C_0805_2012Metric_Pad1.18x1.45mm_HandSolder
- removed D22: 1N5819HW-7-F, EasyEDA:SOD-123_L2.7-W1.6-LS3.7-RD
- removed D27, D28, D29, D30, D31: LESD5D5.0CT1G, EasyEDA:SOD-523_L1.2-W0.8-LS1.6-BI
- removed L1: APH0420T1R0M, EasyEDA:IND-SMD_L4.4-W4.2
- removed LED10, LED11, LED16, LED9: YLED0805G, EasyEDA:LED0805-FD-GREEN
- removed Q13, Q15: 2n3904S-RTK/PS_C18536, EasyEDA:SOT-23-3_L2.9-W1.3-P1.90-LS2.4-TR
- removed R1: 2R, Resistor_SMD:R_0805_2012Metric_Pad1.20x1.40mm_HandSolder
- removed R10: 0.5R, Resistor_SMD:R_0805_2012Metric_Pad1.20x1.40mm_HandSolder
- removed R18, R6: 2.2k, Resistor_SMD:R_0805_2012Metric_Pad1.20x1.40mm_HandSolder
- removed R2: 51k, Resistor_SMD:R_0805_2012Metric_Pad1.20x1.40mm_HandSolder
- removed R3, R4: 100, Resistor_SMD:R_0805_2012Metric_Pad1.20x1.40mm_HandSolder
- removed R74, R75, R9: 1k, Resistor_SMD:R_0805_2012Metric_Pad1.20x1.40mm_HandSolder
- removed RESET1: RESET, EasyEDA:SW-SMD_4P-L6.0-W6.0-P4.50-LS8.2
- removed SGM2212-3.1: ~, Package_TO_SOT_SMD:SOT-223
- removed the THECPCENTER at (241.6, 168.5)
- removed U1: IP2312-4V35, EasyEDA:ESOP-8_L4.9-W3.9-P1.27-LS6.0-BL-EP
- removed U13: ESP32-WROOM-32D, RF_Module:ESP32-WROOM-32D
- removed U14: CH340C, Package_SO:SOIC-16_3.9x9.9mm_P1.27mm
- removed USB2: HX-TYPE-C 16P 180 LT H15.0, EasyEDA:USB-C-SMD_HX-TYPE-C-16P-180-LT-H15.0
- moved D4 0.56 mm to (167.8, 131.8)
- moved SW4 0.10 mm to (134.2, 146.8)
- moved NT1 0.07 mm to (161.9, 196.7)
Connections:
- H2 pad 8: GND -> 3.3V
Routing:
- net GND: track 87.8 -> 106.7 mm, vias 139 -> 143
- net /CC2_1: track 18.2 -> 19.3 mm
- net Net-(C22-Pad1): track 10.2 -> 9.44 mm
- net /V5_1: track 31.4 -> 30.8 mm
- net Net-(D6-A): track 4.15 -> 3.81 mm, vias 3 -> 0
- net Net-(D3-K): vias 9 -> 0
- net /VCC_MOTOR: vias 22 -> 21

Commit message: Update of power desing
Parts:
- added THECPCENTER: LOGO, images:IMG1, F.Cu at (237.3, 166.8)
- R24: footprint Resistor_SMD:R_0805_2012Metric_Pad1.20x1.40mm_HandSolder -> Capacitor_SMD:C_0805_2012Metric_Pad1.18x1.45mm_HandSolder
- moved REF** 16.6 mm to (220.5, 147.9)
- moved R23 13.1 mm to (168.7, 152.8), turned to 90 degrees
- moved C21 9.29 mm to (166.7, 152.8)
- moved R22 7.05 mm to (169.4, 159.2)
- moved USB3 7.05 mm to (173.2, 159.2)
- moved R24 5.34 mm to (170.2, 141.7), turned to 180 degrees
- moved R15 5.10 mm to (169.2, 162.3)
- moved RUN1 5.10 mm to (173.3, 162.2)
- moved U3 3.41 mm to (169.2, 146.7), turned to 0 degrees
- moved 3.3V1 3.12 mm to (173.4, 165.2)
- moved R14 3.12 mm to (169.3, 165.2)
- moved C31 2.36 mm to (165.4, 142.7), turned to -90 degrees
- moved BAT1 1.40 mm to (173.3, 168.5)
- moved R17 1.40 mm to (169.2, 168.5)
- moved R29 0.85 mm to (160.6, 142.8), turned to 180 degrees
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- renumbered H2 to H1.1, H2 to H2.1, H2 to H3.1, H2 to H4.1
Connections:
- H2 pad 8: 3.3V -> GND
Routing:
- net /VDD: track 11.8 -> 0.00 mm
- net /IO19_1: track 41.4 -> 46.7 mm
- net /IO16_1: track 28.7 -> 24.6 mm
- net Net-(U3-VBUS): track 6.07 -> 2.03 mm, vias 2 -> 0
- net 3.3V: track 42.1 -> 38.1 mm
- net /V5_1: track 30.8 -> 33.2 mm, vias 33 -> 32
- net /CC1_1: track 13.4 -> 14.8 mm
- net Net-(D5-C): track 10.8 -> 11.7 mm
- net /CC2_1: track 19.3 -> 18.5 mm
- net /IO17_1: track 98.7 -> 98.1 mm
- net GND: track 106.7 -> 106.8 mm, vias 143 -> 142
- net Net-(C23-Pad1): vias 0 -> 1
- added copper zone on F.Cu, net /VDD
