File: HARDWARE/HydroScan_V1.kicad_pcb (KiCad board)
At the start: 4 copper layers, 222 x 100 mm, 116 parts, among them Q1 AO4435_C2944310, Q14 2n3904S-RTK/PS_C18536, Q16 2n3904S-RTK/PS_C18536, SW2 BOOT, SW4 RESET, U10 DB125-3.81-2P-BK-S, U11 DB125-3.81-2P-BK-S, U15 CH340C, U16 ESP32-WROOM-32D, U2 L298N, U3 CH224K, U4 CN3795, U5 LM358DR, U7 LM2576HVS-3.3, U8 DB125-3.81-2P-BK-S, U9 DB125-3.81-2P-BK-S

Commit message: DRC update
Parts:
- removed 1.1, 1.2 (x3): MountingHole_2.2mm_M2_ISO14580_Pad, MountingHole:MountingHole_2.2mm_M2_ISO14580_Pad
- removed the ? at (293.8, 182.3)
- removed the ? at (188.2, 154.6)
- removed the ? at (293.8, 154.6)
- removed the REF** at (247.7, 159.8)
- added 3.3V2: 3V, TestPoint:TestPoint_Pad_2.5x2.5mm, F.Cu at (193.4, 147.1)
- added 5V1: 5V, TestPoint:TestPoint_Pad_2.5x2.5mm, F.Cu at (252.4, 147.6)
- added ?: , , F.Cu at (285.3, 150.3)
- added ?: , , F.Cu at (285.3, 186.3)
- added ?: , , F.Cu at (260.3, 150.3)
- added ?: , , F.Cu at (260.3, 186.3)
- added C32: 10uf_25v, Capacitor_SMD:C_0805_2012Metric_Pad1.18x1.45mm_HandSolder, F.Cu at (215.2, 148.7)
- added C33: 10uf_25v, Capacitor_SMD:C_0805_2012Metric_Pad1.18x1.45mm_HandSolder, F.Cu at (230.2, 148.9)
- added C34: 10uf_25v, Capacitor_SMD:C_0805_2012Metric_Pad1.18x1.45mm_HandSolder, F.Cu at (237.1, 147.6)
- added C61: 0.1uf, Capacitor_SMD:C_0805_2012Metric_Pad1.18x1.45mm_HandSolder, F.Cu at (230.2, 146.9)
- added C62: 0.1uf, Capacitor_SMD:C_0805_2012Metric_Pad1.18x1.45mm_HandSolder, F.Cu at (215.2, 146.7)
- added C63: 0.1uf, Capacitor_SMD:C_0805_2012Metric_Pad1.18x1.45mm_HandSolder, F.Cu at (245.7, 148.8)
- added DC1: DC-470-2.1GP, EasyEDA:DC-IN-TH_DC-470-2.1GP, F.Cu at (168.7, 170.5)
- added G***: LOGO, EasyEDA:Hydroscan1, F.Cu at (232.0, 168.7)
- added GND2: GND, TestPoint:TestPoint_Pad_2.5x2.5mm, F.Cu at (291.4, 191.3)
- added H5: 2.54-2*10, EasyEDA:HDR-TH_20P-P2.54-V-M-R2-C10-S2.54, F.Cu at (242.6, 190.1)
- added J1: Conn_01x08_Pin, EasyEDA:MPU6050_Module, B.Cu at (243.8, 159.8)
- added J2: Conn_01x03_Pin, Connector_PinHeader_2.54mm:PinHeader_1x03_P2.54mm_Vertical, B.Cu at (214.2, 159.5)
- added JP1: SolderJumper_3_Open, Jumper:SolderJumper-3_P1.3mm_Open_RoundedPad1.0x1.5mm_NumberLabels, F.Cu at (224.3, 159.5)
- added JP2: SolderJumper_2_Open, Jumper:SolderJumper-2_P1.3mm_Open_Pad1.0x1.5mm, F.Cu at (242.5, 182.9)
- added R37: 4.7K, Resistor_SMD:R_0805_2012Metric_Pad1.20x1.40mm_HandSolder, F.Cu at (205.3, 186.6)
- added R38: 4.7K, Resistor_SMD:R_0805_2012Metric_Pad1.20x1.40mm_HandSolder, F.Cu at (214.2, 186.6)
- added R40: 6.8k, Resistor_SMD:R_0805_2012Metric_Pad1.20x1.40mm_HandSolder, F.Cu at (245.7, 146.8)
- added REF**: MountingHole_2.2mm_M2_DIN965_Pad_TopBottom, MountingHole:MountingHole_2.2mm_M2_DIN965_Pad_TopBottom, F.Cu at (188.2, 154.6)
- added REF**: MountingHole_2.2mm_M2_DIN965_Pad_TopBottom, MountingHole:MountingHole_2.2mm_M2_DIN965_Pad_TopBottom, F.Cu at (188.2, 182.3)
- added REF**: MountingHole_2.2mm_M2_DIN965_Pad_TopBottom, MountingHole:MountingHole_2.2mm_M2_DIN965_Pad_TopBottom, F.Cu at (293.8, 182.3)
- added REF**: MountingHole_2.2mm_M2_DIN965_Pad_TopBottom, MountingHole:MountingHole_2.2mm_M2_DIN965_Pad_TopBottom, F.Cu at (293.8, 154.6)
- added THECPCENTER: LOGO, images:IMG1, F.Cu at (193.9, 189.9)
- added U1: SY6280AAC, EasyEDA:SOT-23-5_L3.0-W1.7-P0.95-LS2.8-BL, F.Cu at (241.4, 147.4)
- added _: modulo esp32, EasyEDA:modulo esp32, F.Cu at (264.4, 175.8)
- moved H4 31.2 mm to (222.7, 147.9)
- moved 1A 4.20 mm to (109.6, 143.6)
- moved 3.3V1 2.34 mm to (173.2, 162.9)
- moved BAT1 2.34 mm to (173.2, 166.1)
- moved R14 2.34 mm to (169.2, 163.0)
- moved R15 2.34 mm to (169.1, 160.0)
- moved R17 2.34 mm to (169.1, 166.1)
- moved R22 2.34 mm to (169.3, 156.9)
- moved RUN1 2.34 mm to (173.2, 159.9)
- moved USB3 2.34 mm to (173.1, 156.9)
- moved REF** 1.39 mm to (166.1, 124.8)
- moved C25 0.67 mm to (175.3, 183.0)
- moved C29 0.62 mm to (158.6, 178.6)
- moved C27 0.48 mm to (174.6, 190.0)
- moved D5 0.40 mm to (163.7, 164.9)
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- renumbered G*** to 1A
Connections:
- H1 pad 16: /V_BAT -> /BAT_2_1
- H3 pad 11: /IO38 -> /INT
- H4 pad 1: unconnected-(H4-Pad1) -> 3.3V+
- H4 pad 2: unconnected-(H4-Pad2) -> GND
- H4 pad 3: unconnected-(H4-Pad3) -> GND
- H4 pad 4: unconnected-(H4-Pad4) -> /OUT_PUT_ UP
Routing:
- net /IO9: track 0.00 -> 77.3 mm
- net /IO5: track 0.00 -> 66.8 mm, vias 0 -> 2
- net /IO8: track 0.00 -> 59.2 mm
- net /IO1: track 0.00 -> 53.2 mm
- net /BAT_2: track 0.00 -> 39.2 mm, vias 0 -> 18
- net /IO12: track 0.00 -> 31.0 mm
- net /IO11: track 0.00 -> 30.0 mm
- net /IO10: track 0.00 -> 30.0 mm
- net /INT: track 0.00 -> 28.9 mm
- net GND: track 108.1 -> 135.5 mm, vias 136 -> 164
- net /V5_1: track 25.3 -> 7.87 mm
- net /IO2: track 0.00 -> 16.9 mm
- net /BAT_2_1: track 0.00 -> 11.8 mm
- net 3.3V+: track 0.00 -> 11.3 mm, vias 0 -> 6
- net Net-(J2-Pin_2): track 0.00 -> 10.2 mm
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- added copper zone on In2.Cu, net +5V
- added copper zone on B.Cu, net /BAT_2
- added copper zone on F.Cu, net /BAT_2
- added copper zone on In2.Cu, net /BAT_2
- added copper zone on F.Cu, net /OUT_PUT_ UP
- added copper zone on In2.Cu, net 3.3V+
- removed copper zone on B.Cu, net /VCC_MOTOR
Other:
- outline, holes or cut-outs redrawn
- board text added: "TDS METER V1"

Commit message: PCB_v1
manufacturing list
Parts:
- removed the H4 at (222.7, 147.9)
- added 3.3V3: TestPoint, TestPoint:TestPoint_Pad_2.0x2.0mm, F.Cu at (82.4, 177.2)
- added BATTERY1: TestPoint, TestPoint:TestPoint_Pad_2.0x2.0mm, F.Cu at (157.9, 217.3)
- added C64: 0.1uf, Capacitor_SMD:C_0805_2012Metric_Pad1.18x1.45mm_HandSolder, B.Cu at (203.9, 150.3)
- added DC_BOOST_1: PZ254V-11-04P_C2691448, EasyEDA:HDR-TH_4P-P2.54-V-M, F.Cu at (238.2, 147.2)
- added GND3: TestPoint, TestPoint:TestPoint_Pad_2.0x2.0mm, F.Cu at (152.5, 217.3)
- added JP3: SolderJumper_3_Open, Jumper:SolderJumper-3_P1.3mm_Open_RoundedPad1.0x1.5mm_NumberLabels, B.Cu at (248.5, 177.5)
- added JP4: SolderJumper_2_Open, Jumper:SolderJumper-2_P1.3mm_Open_Pad1.0x1.5mm, F.Cu at (217.8, 149.7)
- added JP5: SolderJumper_2_Open, Jumper:SolderJumper-2_P1.3mm_Open_Pad1.0x1.5mm, F.Cu at (181.2, 169.3)
- added R39: 100K, Resistor_SMD:R_0805_2012Metric_Pad1.20x1.40mm_HandSolder, B.Cu at (248.4, 182.4)
- added R41: 100K, Resistor_SMD:R_0805_2012Metric_Pad1.20x1.40mm_HandSolder, B.Cu at (248.4, 184.4)
- added USB2: TestPoint, TestPoint:TestPoint_Pad_2.0x2.0mm, F.Cu at (177.5, 151.3)
- JP1: moved to B.Cu
- moved REF** 49.4 mm to (290.8, 147.2)
- moved R40 23.8 mm to (221.9, 145.8)
- moved C34 23.8 mm to (213.3, 146.6)
- moved C63 23.8 mm to (221.9, 147.9)
- moved U1 23.8 mm to (217.6, 146.5)
- moved C62 15.6 mm to (230.8, 145.9)
- moved C61 15.6 mm to (245.8, 145.9)
- moved C33 15.6 mm to (245.8, 148.0)
- moved C32 15.6 mm to (230.8, 148.0)
- moved JP1 3.08 mm to (223.8, 156.5), turned to 0 degrees
- moved USB3 0.37 mm to (173.5, 157.0)
- moved RUN1 0.30 mm to (173.5, 160.0)
- moved BAT1 0.26 mm to (173.5, 166.2)
- moved 3.3V1 0.24 mm to (173.5, 162.9)
- turned H7.1 to -90 degrees
- gave numbers to parts that had none: 4
- renumbered H1 to H5.1, H3 to H5.2, REF** to H8.1, REF** to H8.2, REF** to H8.3, REF** to H8.4
Connections:
- net /VCC_MOTOR renamed V_BATTERY__1
- C32 pad 1: 3.3V+ -> 3.3V+_1
- C33 pad 1: /OUT_PUT_ UP -> +5V
- C34 pad 1: /OUT_PUT_ UP -> 3.3V+
- C61 pad 2: /OUT_PUT_ UP -> +5V
- C62 pad 2: 3.3V+ -> 3.3V+_1
- C63 pad 2: +5V -> 3.3V+_1
- H5 pad 10: unconnected-(H5-Pad10) -> /IO48
- H5 pad 13: unconnected-(H5-Pad13) -> 3.3V+_1
- H5 pad 14: unconnected-(H5-Pad14) -> 3.3V+_1
- H5 pad 7: /IO1 -> /UART0_TX
- H5 pad 9: unconnected-(H5-Pad9) -> /UART0_RX
- H7.1 pad 1: (no net) -> GND
- H7.2 pad 1: (no net) -> GND
- H7.3 pad 1: (no net) -> GND
- H7.4 pad 1: (no net) -> GND
- H8.2 pad 1: (no net) -> GND
- H8.3 pad 1: (no net) -> GND
- J1 pad 8: 3.3V+ -> Net-(J1-Pin_8)
- JP1 pad 1: 3.3V+ -> 3.3V+_1
- U1 pad 1: +5V -> 3.3V+_1
- U1 pad 5: /OUT_PUT_ UP -> 3.3V+
- U16 pad 6: /IO34_1 -> unconnected-(U16-IO34-Pad6)
- U16 pad 7: /IO35_1 -> unconnected-(U16-IO35-Pad7)
Routing:
- net /UART0_RX: track 0.00 -> 64.7 mm, vias 0 -> 1
- net /UART0_TX: track 0.00 -> 63.8 mm, vias 0 -> 1
- net +5V: track 9.68 -> 35.4 mm, vias 9 -> 6
- net /IO48: track 0.00 -> 23.8 mm
- net /IO5: track 66.8 -> 46.1 mm
- net /IO1: track 53.2 -> 64.7 mm
- net 3.3V+_1: track 0.00 -> 8.20 mm, vias 0 -> 11
- net Net-(J1-Pin_8): track 0.00 -> 7.42 mm
- net /OUT_PUT_ UP: track 6.73 -> 0.00 mm
- net /BAT_2: track 39.2 -> 45.2 mm, vias 18 -> 19
- net 3.3V+: track 11.3 -> 5.73 mm, vias 6 -> 11
- net /V5_1: track 7.87 -> 12.7 mm, vias 29 -> 31
- net V_BATTERY__1: track 59.4 -> 62.2 mm, vias 15 -> 17
- net 3.3V: track 38.9 -> 41.1 mm, vias 29 -> 31
- net GND: track 135.5 -> 133.6 mm, vias 164 -> 167
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- added copper zone on F.Cu, net 3.3V+
- added copper zone on F.Cu, net 3.3V+_1
- added copper zone on In2.Cu, net 3.3V+_1
- removed copper zone on F.Cu, net /OUT_PUT_ UP
Other:
- board text added: "BATTERY"
- board text removed: "BATERY"

Commit message: BOM generate
Parts:
- added BATTERY2: TestPoint, TestPoint:TestPoint_Pad_2.0x2.0mm, F.Cu at (147.1, 217.3)
- added JP6: SolderJumper_3_Open, Jumper:SolderJumper-3_P1.3mm_Open_RoundedPad1.0x1.5mm_NumberLabels, B.Cu at (157.4, 121.9)
- added JP7: SolderJumper_3_Open, Jumper:SolderJumper-3_P1.3mm_Open_RoundedPad1.0x1.5mm_NumberLabels, B.Cu at (123.5, 132.8)
- added R1: TC33X-2-103E, EasyEDA:RES-ADJ-SMD_3P-L3.0-W3.8-P1.75-BR, F.Cu at (252.5, 146.7)
- added R42: 10k, Resistor_SMD:R_0805_2012Metric_Pad1.20x1.40mm_HandSolder, F.Cu at (152.7, 121.5)
- added R43: 10k, Resistor_SMD:R_0805_2012Metric_Pad1.20x1.40mm_HandSolder, F.Cu at (128.6, 130.6)
- added TP1: TDS_1, TestPoint:TestPoint_THTPad_D4.0mm_Drill2.0mm, F.Cu at (277.2, 152.7)
- added TP2: TDS_2, TestPoint:TestPoint_THTPad_D4.0mm_Drill2.0mm, F.Cu at (264.4, 145.9)
- moved 5V1 12.7 mm to (240.9, 153.1)
- moved R34 1.09 mm to (128.6, 134.7)
- moved R33 1.02 mm to (128.6, 132.6)
- moved R28 0.42 mm to (152.7, 129.4)
- moved R32 0.42 mm to (152.8, 123.5)
- moved R81 0.39 mm to (152.7, 127.5)
- moved Q14 0.38 mm to (154.2, 132.5)
- moved R82 0.36 mm to (152.7, 125.5)
- moved R80 0.28 mm to (153.8, 136.6)
- moved C59 0.23 mm to (128.6, 126.4)
- moved JP4 0.17 mm to (217.8, 149.9)
- moved C60 0.16 mm to (128.5, 128.5)
Connections:
- U16 pad 29: /IO5_1 -> unconnected-(U16-IO5-Pad29)
Routing:
- net Net-(R1-Pad1): track 0.00 -> 25.2 mm
- net Net-(R1-Pad2): track 0.00 -> 15.3 mm
- net Net-(JP6-C): track 0.00 -> 6.50 mm, vias 0 -> 1
- net Net-(JP7-C): track 0.00 -> 5.38 mm, vias 0 -> 1
- net /IO23_1: track 67.4 -> 70.6 mm
- net /VN_1: track 39.4 -> 36.4 mm
- net GND: track 133.6 -> 135.2 mm, vias 167 -> 169
- net /IO32_1: track 56.1 -> 57.4 mm
- net V_BATTERY__1: track 62.2 -> 63.5 mm, vias 17 -> 19
- net /IO13_1: track 57.6 -> 58.8 mm
- net /IO25_1: track 82.8 -> 83.3 mm
- net 3.3V: track 41.1 -> 40.6 mm, vias 31 -> 33
Other:
- board text added: "BATTERY1"
